File: kiCad/LineSensor_Prot2/LineSensor.kicad_sch (KiCad schematic)
At the start: 98 parts, among them J1 Conn_01x07_Socket, J2 Conn_01x07_Socket, J3 Conn_01x07_Socket, J4 Conn_01x07_Socket, Q1 Q_Photo_NPN, Q10 Q_Photo_NPN, Q11 Q_Photo_NPN, Q12 Q_Photo_NPN, Q13 Q_Photo_NPN, Q14 Q_Photo_NPN, Q15 Q_Photo_NPN, Q16 Q_Photo_NPN, Q2 Q_Photo_NPN, Q3 Q_Photo_NPN, Q4 Q_Photo_NPN, Q5 Q_Photo_NPN, Q6 Q_Photo_NPN, Q7 Q_Photo_NPN, Q8 Q_Photo_NPN, Q9 Q_Photo_NPN, U1 LM393, U10 LM393, U11 LM393, U12 LM393, U2 LM393, U3 LM393, U4 LM393, U5 LM393, U6 LM393, U7 LM393, U8 LM393, U9 LM393

Commit message: 30
Parts:
- removed C1: C, Capacitor_THT:C_Disc_D7.0mm_W2.5mm_P5.00mm, symbol Device:C
- removed J1, J2, J3, J4: Conn_01x07_Socket, symbol Connector:Conn_01x07_Socket
- removed unit 3 of U1
- removed U10, U11, U12, U9: LM393, Package_DIP:DIP-8_W7.62mm_Socket_LongPads, symbol Comparator:LM393
- added C10, C11, C4, C5, C6, C7, C8, C9: C, Capacitor_THT:C_Disc_D7.0mm_W2.5mm_P5.00mm, symbol Device:C
- added C2, C3: C, symbol Device:C
- added D17: D, symbol Device:D
- added D18, D19, D20, D21, D22, D23, D24, D25, D26, D27, D28, D29, D30, D31, D32, D33, D34, D35, D36, D37, D38, D39, D40, D41, D42, D43, D44, D45, D46, D47, D48, D49: LED, LED_THT:LED_D3.0mm, symbol Device:LED
- added F2: Polyfuse, symbol Device:Polyfuse
- added J1: Conn_01x04_Socket, symbol Connector:Conn_01x04_Socket
- added J2: Conn_01x02_Socket, symbol Connector:Conn_01x02_Socket
- added R49, R50, R51: R, symbol Device:R
- added R52, R53, R54, R55, R56, R57, R58, R59, R60, R61, R62, R63, R64, R65, R66, R67, R68, R69, R70, R71, R72, R73, R74, R75, R76, R77, R78, R79, R80, R81, R82, R83: R, Resistor_THT:R_Axial_DIN0207_L6.3mm_D2.5mm_P7.62mm_Horizontal, symbol Device:R
- added RV1, RV2, RV3, RV4: R_Potentiometer_Trim, symbol Device:R_Potentiometer_Trim
- added SW2: SW_DPST_x2, symbol Switch:SW_DPST_x2
- added unit 1 of U2
- added unit 3 of U2
- added unit 3 of U3
- added unit 1 of U3
- added unit 3 of U4
- added unit 1 of U5
- added unit 3 of U5
- added unit 3 of U6
- added unit 1 of U6
- added unit 3 of U7
- added unit 1 of U8
- added unit 3 of U8
- added U9: LM393, symbol Comparator:LM393
- U1, U2, U3, U4, U5, U6, U7, U8: footprint Package_DIP:DIP-8_W7.62mm_Socket_LongPads -> (none)
Connections:
- net GND: now also R13.2, R14.2, R15.2, R16.2, R25.2, R26.2, R27.2, R28.2, R37.2, R38.2, R39.2, R40.2, R5.2, R6.2, C10.2, C11.2, C2.1, C3.2, C4.2, C5.2, C6.2, C7.2, C8.2, C9.2, D17.1 (K), J1.3 (Pin_3), J2.2 (Pin_2), R50.2, RV1.3, RV2.3, RV3.3, RV4.3, U2.8 (V+), U3.8 (V+), U4.8 (V+), U5.8 (V+), U6.4 (V-), U7.4 (V-), U8.4 (V-), U9.4 (V-); no longer R10.2, R21.2, R22.2, R23.2, R24.2, R33.2, R34.2, R35.2, R36.2, R45.2, R46.2, R47.2, R48.2, R9.2
- net VCC: now also R10.1, R21.1, R22.1, R23.1, R24.1, R33.1, R34.1, R35.1, R36.1, R45.1, R46.1, R47.1, R48.1, R9.1, C10.1, C11.1, C2.2, C3.1, C4.1, C5.1, C6.1, C7.1, C8.1, C9.1, D17.2 (A), F2.2, RV1.1, RV2.1, RV3.1, RV4.1, SW2.1 (A), U2.4 (V-), U3.4 (V-), U4.4 (V-), U5.4 (V-), U6.8 (V+), U7.8 (V+), U8.8 (V+), U9.8 (V+); no longer R13.1, R14.1, R15.1, R16.1, R25.1, R26.1, R27.1, R28.1, R37.1, R38.1, R39.1, R40.1, R5.1, R6.1
- net at D9.1 (K): now also R25.1; no longer R33.1
- net at R3.1: now also Q3.2 (E), U4.3 (+); no longer D1.1 (K)
- net at U7.3 (+), U7.5 (+), U8.5 (+): now also RV3.2, U8.3 (+)
- net at Q12.2 (E), R32.1: now also U5.3 (+)
- net at R11.2: now also A1.11 (D8), U4.1; no longer U2.7
- net at Q5.2 (E), R17.1: now also U8.6 (-); no longer U4.2 (-)
- net at Q10.2 (E), R30.1: now also U6.3 (+); no longer U7.6 (-)
- net at U7.7: now also A1.21 (A2), R23.2; no longer R26.2
- net at U4.7: now also A1.12 (D9), R12.2; no longer R14.2
- net at U5.7: now also A1.7 (D4), R35.2; no longer R15.2
- net at U6.7: now also A1.5 (D2), R33.2; no longer R16.2
- net at Q9.2 (E), R29.1: now also U6.5 (+); no longer U7.2 (-)
- net at Q1.2 (E), R1.1: now also U3.3 (+); no longer U1.2 (-)
- net at D7.1 (K): now also R15.1; no longer R23.1
- net at Q16.2 (E), R44.1: now also U2.5 (+)
- net at R4.1: now also Q4.2 (E), U4.5 (+); no longer D2.1 (K)
- net at Q11.2 (E), R31.1: now also U5.5 (+); no longer U8.6 (-)
- net at U8.7: now also A1.19 (A0), R21.2; no longer R27.2
- net at Q8.2 (E), R20.1: now also U7.2 (-); no longer U6.6 (-)
- net at D6.1 (K): now also R14.1; no longer R22.1
- net at Q2.2 (E), R2.1: now also U3.5 (+); no longer U1.6 (-)
- net at U1.7: now also A1.14 (D11), R46.2; no longer R6.2
- net at U7.1: now also A1.22 (A3), R24.2; no longer R25.2
- net at D16.1 (K): now also R40.1; no longer R48.1
- net at Q13.2 (E), R41.1: now also U1.3 (+)
- net at U1.1: now also A1.13 (D10), R45.2; no longer R5.2
- net at U3.7: now also A1.10 (D7), R10.2; no longer R12.2
- net at Q7.2 (E), R19.1: now also U7.6 (-); no longer U5.6 (-)
- net at Q6.2 (E), R18.1: now also U8.2 (-); no longer U4.6 (-)
- net at A1.1 (D1/TX): now also R49.2
- net at A1.15 (D12): now also R47.2
- net at A1.16 (D13): now also R48.2, U2.7
- net at A1.2 (D0/RX): now also J1.2 (Pin_2)
- net at A1.20 (A1): now also R22.2, U8.1
- net at A1.6 (D3): now also R34.2, U6.1
- net at A1.8 (D5): now also R36.2, U5.1
- net at A1.9 (D6): now also R9.2, U3.1
- net at D14.1 (K): now also R38.1; no longer R46.1
- net at Q14.2 (E), R42.1: now also U1.5 (+)
- net at D8.1 (K): now also R16.1; no longer R24.1
- net at D12.1 (K): now also R28.1; no longer R36.1
- net at D5.1 (K): now also R13.1; no longer R21.1
- net at D13.1 (K): now also R37.1; no longer R45.1
- net at D10.1 (K): now also R26.1; no longer R34.1
- net at D11.1 (K): now also R27.1; no longer R35.1
- net at D15.1 (K): now also R39.1; no longer R47.1
- new net: J1.1 (Pin_1), R49.1, R51.1
- new net: D27.1 (K), R61.1
- new net: R52.2, R53.2, R54.2, R55.2, R56.2, R57.2, R58.2, R59.2, R60.2, R61.2, R62.2, R63.2, R64.2, R65.2, R66.2, R67.2, R68.2, R69.2, R70.2, R71.2, R72.2, R73.2, R74.2, R75.2, R76.2, R77.2, R78.2, R79.2, R80.2, R81.2, R82.2, R83.2
- new net: D46.1 (K), R80.1
- new net: D18.2 (A), D19.2 (A), D20.2 (A), D21.2 (A), D22.2 (A), D23.2 (A), D24.2 (A), D25.2 (A), D26.2 (A), D27.2 (A), D28.2 (A), D29.2 (A), D30.2 (A), D31.2 (A), D32.2 (A), D33.2 (A), D34.2 (A), D35.2 (A), D36.2 (A), D37.2 (A), D38.2 (A), D39.2 (A), D40.2 (A), D41.2 (A), D42.2 (A), D43.2 (A), D44.2 (A), D45.2 (A), D46.2 (A), D47.2 (A), D48.2 (A), D49.2 (A)
- new net: D45.1 (K), R79.1
- new net: D30.1 (K), R64.1
- new net: D21.1 (K), R55.1
- new net: D43.1 (K), R77.1
- new net: D33.1 (K), R67.1
- new net: RV2.2, U5.2 (-), U5.6 (-), U6.2 (-), U6.6 (-)
- new net: D23.1 (K), R57.1
- new net: D26.1 (K), R60.1
- new net: R50.1, R51.2
- new net: D39.1 (K), R73.1
- new net: RV1.2, U3.2 (-), U3.6 (-), U4.2 (-), U4.6 (-)
- new net: D36.1 (K), R70.1
- new net: D42.1 (K), R76.1
- new net: D20.1 (K), R54.1
- new net: D32.1 (K), R66.1
- new net: D29.1 (K), R63.1
- new net: RV4.2, U1.2 (-), U1.6 (-), U2.6 (-)
- new net: D2.1 (K), R6.1
- new net: D49.1 (K), R83.1
- new net: D37.1 (K), R71.1
- new net: D28.1 (K), R62.1
- new net: J2.1 (Pin_1), SW2.2 (B)
- new net: D1.1 (K), R5.1
- new net: D35.1 (K), R69.1
- new net: D18.1 (K), R52.1
- new net: F2.1, J1.4 (Pin_4)
- new net: D22.1 (K), R56.1
- new net: D34.1 (K), R68.1
- new net: D38.1 (K), R72.1
- new net: D25.1 (K), R59.1
- new net: D31.1 (K), R65.1
- new net: D48.1 (K), R82.1
- new net: D19.1 (K), R53.1
- new net: D24.1 (K), R58.1
- new net: D41.1 (K), R75.1
- new net: D47.1 (K), R81.1
- new net: D40.1 (K), R74.1
- new net: D44.1 (K), R78.1
Other:
- note removed: "atmega328"
- moved on the sheet: A1

Commit message: フットプリント割あて.25.11.3
Parts:
- removed D1, D10, D11, D12, D13, D14, D15, D16, D2, D3, D4, D5, D6, D7, D8, D9: LED, LED_THT:LED_D3.0mm, symbol Device:LED
- removed F2: Polyfuse, symbol Device:Polyfuse
- removed R1, R10, R11, R12, R13, R14, R15, R16, R17, R18, R19, R2, R20, R21, R22, R23, R24, R25, R26, R27, R28, R29, R3, R30, R31, R32, R33, R34, R35, R36, R37, R38, R39, R4, R40, R41, R42, R43, R44, R45, R46, R47, R48, R5, R52, R53, R54, R55, R56, R57, R58, R59, R6, R60, R61, R62, R63, R64, R65, R66, R67, R68, R69, R7, R70, R71, R72, R73, R74, R75, R76, R77, R78, R79, R8, R80, R81, R82, R83, R9: R, Resistor_THT:R_Axial_DIN0207_L6.3mm_D2.5mm_P7.62mm_Horizontal, symbol Device:R
- added Q17: NMOS, Package_TO_SOT_THT:TO-251-3-1EP_Horizontal_TabDown, symbol Simulation_SPICE:NMOS
- added R84, R85: R, Resistor_THT:R_Axial_DIN0207_L6.3mm_D2.5mm_P7.62mm_Horizontal, symbol Device:R
- added RN1, RN10, RN11, RN12, RN13, RN14, RN15, RN16, RN2, RN3, RN4, RN5, RN6, RN7, RN8, RN9: R_Network04, Resistor_SMD:R_Array_Convex_4x1206, symbol Device:R_Network04
- C10, C11, C4, C5, C6, C7, C8, C9: footprint Capacitor_THT:C_Disc_D7.0mm_W2.5mm_P5.00mm -> Capacitor_SMD:C_0603_1608Metric
- C2: footprint (none) -> Capacitor_THT:CP_Radial_Tantal_D5.0mm_P5.00mm
- C3: footprint (none) -> Capacitor_THT:C_Radial_D6.3mm_H11.0mm_P2.50mm
- D17: footprint (none) -> Diode_THT:D_DO-201AD_P12.70mm_Horizontal
- D18, D19, D20, D21, D22, D23, D24, D25, D26, D27, D28, D29, D30, D31, D32, D33, D34, D35, D36, D37, D38, D39, D40, D41, D42, D43, D44, D45, D46, D47, D48, D49, Q1, Q10, Q11, Q12, Q13, Q14, Q15, Q16, Q2, Q3, Q4, Q5, Q6, Q7, Q8, Q9: footprint LED_THT:LED_D3.0mm -> LED_SMD:LED_0603_1608Metric
- J1: footprint (none) -> Connector_PinSocket_2.54mm:PinSocket_1x04_P2.54mm_Vertical
- J2: footprint (none) -> Connector_PinSocket_2.54mm:PinSocket_1x02_P2.54mm_Vertical
- R49, R50, R51: footprint (none) -> Resistor_THT:R_Axial_DIN0207_L6.3mm_D2.5mm_P7.62mm_Horizontal
- RV1, RV2, RV3, RV4: footprint (none) -> Connector_PinHeader_2.54mm:PinHeader_1x03_P2.54mm_Vertical
- SW2: footprint (none) -> Connector_PinSocket_2.54mm:PinSocket_1x03_P2.54mm_Vertical
- U1, U2, U3, U4, U5, U6, U7, U8, U9: footprint (none) -> Package_SO:SOIC-8_3.9x4.9mm_P1.27mm
Connections:
- net GND: now also Q17.3 (S), R85.1, RN13.1 (common), RN14.1 (common), RN15.1 (common), RN16.1 (common)
- net VCC: now also D18.2 (A), D19.2 (A), D20.2 (A), D21.2 (A), D22.2 (A), D23.2 (A), D24.2 (A), D25.2 (A), D26.2 (A), D27.2 (A), D28.2 (A), D29.2 (A), D30.2 (A), D31.2 (A), D32.2 (A), D33.2 (A), D34.2 (A), D35.2 (A), D36.2 (A), D37.2 (A), D38.2 (A), D39.2 (A), D40.2 (A), D41.2 (A), D42.2 (A), D43.2 (A), D44.2 (A), D45.2 (A), D46.2 (A), D47.2 (A), D48.2 (A), D49.2 (A), J1.4 (Pin_4), RN10.1 (common), RN11.1 (common), RN12.1 (common), RN9.1 (common)
- net at Q4.2 (E), U4.5 (+): now also RN15.2 (R1)
- net at Q3.2 (E), U4.3 (+): now also RN15.3 (R2)
- net at A1.15 (D12): now also U1.7, RN9.3 (R2)
- net at Q5.2 (E), U8.6 (-): now also RN13.2 (R1)
- net at D27.1 (K): now also RN3.4 (R3)
- net at Q9.2 (E), U6.5 (+): now also RN16.5 (R4)
- net at A1.5 (D2), U6.7: now also RN11.2 (R1)
- net at D46.1 (K): now also RN8.5 (R4)
- net at D45.1 (K): now also RN7.2 (R1)
- net at A1.13 (D10): now also R84.1; no longer U1.1
- net at A1.11 (D8), U4.1: now also RN12.4 (R3)
- net at D30.1 (K): now also RN4.5 (R4)
- net at D21.1 (K): now also RN1.2 (R1)
- net at Q14.2 (E), U1.5 (+): now also RN14.4 (R3)
- net at D43.1 (K): now also RN7.4 (R3)
- net at D33.1 (K): now also RN4.2 (R1)
- net at A1.8 (D5), U5.1: now also RN11.5 (R4)
- net at Q12.2 (E), U5.3 (+): now also RN16.2 (R1)
- net at Q6.2 (E), U8.2 (-): now also RN13.3 (R2)
- net at Q2.2 (E), U3.5 (+): now also RN15.4 (R3)
- net at U2.1: now also A1.16 (D13), RN9.4 (R3)
- net at U2.2 (-): now also RV4.2, U1.2 (-), U1.6 (-), U2.6 (-)
- net at U2.3 (+): now also Q15.2 (E), RN14.3 (R2)
- net at D23.1 (K): now also RN2.4 (R3)
- net at D26.1 (K): now also RN3.5 (R4)
- net at Q10.2 (E), U6.3 (+): now also RN16.4 (R3)
- net at A1.19 (A0), U8.7: now also RN10.5 (R4)
- net at D39.1 (K): now also RN6.4 (R3)
- net at Q8.2 (E), U7.2 (-): now also RN13.5 (R4)
- net at Q13.2 (E), U1.3 (+): now also RN14.5 (R4)
- net at D36.1 (K): now also RN5.3 (R2)
- net at D42.1 (K): now also RN7.5 (R4)
- net at Q1.2 (E), U3.3 (+): now also RN15.5 (R4)
- net at A1.10 (D7), U3.7: now also RN12.3 (R2)
- net at A1.12 (D9), U4.7: now also RN12.5 (R4)
- net at A1.14 (D11): now also U1.1, RN9.2 (R1); no longer U1.7
- net at U2.7: now also A1.23 (A4), RN9.5 (R4); no longer A1.16 (D13)
- net at A1.20 (A1), U8.1: now also RN10.4 (R3)
- net at A1.21 (A2), U7.7: now also RN10.3 (R2)
- net at A1.22 (A3), U7.1: now also RN10.2 (R1)
- net at A1.6 (D3), U6.1: now also RN11.3 (R2)
- net at A1.7 (D4), U5.7: now also RN11.4 (R3)
- net at A1.9 (D6), U3.1: now also RN12.2 (R1)
- net at D20.1 (K): now also RN1.3 (R2)
- net at D32.1 (K): now also RN4.3 (R2)
- net at Q16.2 (E), U2.5 (+): now also RN14.2 (R1)
- net at D29.1 (K): now also RN3.2 (R1)
- net at D49.1 (K): now also RN8.2 (R1)
- net at D37.1 (K): now also RN5.2 (R1)
- net at D28.1 (K): now also RN3.3 (R2)
- net at Q11.2 (E), U5.5 (+): now also RN16.3 (R2)
- net at D35.1 (K): now also RN5.4 (R3)
- net at D18.1 (K): now also RN1.5 (R4)
- net at Q7.2 (E), U7.6 (-): now also RN13.4 (R3)
- net at D22.1 (K): now also RN2.5 (R4)
- net at D34.1 (K): now also RN5.5 (R4)
- net at D38.1 (K): now also RN6.5 (R4)
- net at D25.1 (K): now also RN2.2 (R1)
- net at D31.1 (K): now also RN4.4 (R3)
- net at D48.1 (K): now also RN8.3 (R2)
- net at D19.1 (K): now also RN1.4 (R3)
- net at D24.1 (K): now also RN2.3 (R2)
- net at D41.1 (K): now also RN6.2 (R1)
- net at D47.1 (K): now also RN8.4 (R3)
- net at D40.1 (K): now also RN6.3 (R2)
- net at D44.1 (K): now also RN7.3 (R2)
- new net: Q17.1 (D), RN1.1 (common), RN2.1 (common), RN3.1 (common), RN4.1 (common), RN5.1 (common), RN6.1 (common), RN7.1 (common), RN8.1 (common)
- new net: Q17.2 (G), R84.2, R85.2
Other:
- moved on the sheet: U2A
