File: kiCad/LineSensor_Prot2/LineSensor.kicad_pcb (KiCad board)
At the start: 2 copper layers, 45.7 x 22.9 mm, 13 parts, among them J1 Conn_01x05_Socket, Q1 Q_Photo_NPN, Q2 Q_Photo_NPN, U1 LM393

Commit message: フットプリント割あて.25.11.3
Parts:
- removed C1: C, Capacitor_THT:C_Disc_D7.0mm_W2.5mm_P5.00mm
- removed D1, D2: LED, LED_THT:LED_D3.0mm
- removed R1, R2, R3, R4, R5, R6: R, Resistor_THT:R_Axial_DIN0207_L6.3mm_D2.5mm_P7.62mm_Horizontal
- added A1: Arduino_Nano_v2.x, Module:Arduino_Nano, F.Cu at (156.7, 44.1)
- added C10: C, Capacitor_SMD:C_0603_1608Metric, F.Cu at (175.8, 65.8)
- added C11: C, Capacitor_SMD:C_0603_1608Metric, F.Cu at (175.8, 69.9)
- added C2: C, Capacitor_THT:CP_Radial_Tantal_D5.0mm_P5.00mm, F.Cu at (184.3, 56.7)
- added C3: C, Capacitor_THT:C_Radial_D6.3mm_H11.0mm_P2.50mm, F.Cu at (193.7, 56.4)
- added C4: C, Capacitor_SMD:C_0603_1608Metric, F.Cu at (175.8, 41.5)
- added C5: C, Capacitor_SMD:C_0603_1608Metric, F.Cu at (175.8, 45.6)
- added C6: C, Capacitor_SMD:C_0603_1608Metric, F.Cu at (175.8, 49.6)
- added C7: C, Capacitor_SMD:C_0603_1608Metric, F.Cu at (175.8, 53.7)
- added C8: C, Capacitor_SMD:C_0603_1608Metric, F.Cu at (175.8, 57.7)
- added C9: C, Capacitor_SMD:C_0603_1608Metric, F.Cu at (175.8, 61.8)
- added D17: D, Diode_THT:D_DO-201AD_P12.70mm_Horizontal, F.Cu at (128.5, 121.4)
- added D18: LED, LED_SMD:LED_0603_1608Metric, F.Cu at (222.5, 117.8)
- added D19: LED, LED_SMD:LED_0603_1608Metric, F.Cu at (222.5, 120.4)
- added D20: LED, LED_SMD:LED_0603_1608Metric, F.Cu at (222.5, 123.0)
- added D21: LED, LED_SMD:LED_0603_1608Metric, F.Cu at (222.5, 125.5)
- added D22: LED, LED_SMD:LED_0603_1608Metric, F.Cu at (222.5, 128.1)
- added D23: LED, LED_SMD:LED_0603_1608Metric, F.Cu at (222.5, 130.7)
- added D24: LED, LED_SMD:LED_0603_1608Metric, F.Cu at (222.5, 133.3)
- added D25: LED, LED_SMD:LED_0603_1608Metric, F.Cu at (222.5, 135.9)
- added D26: LED, LED_SMD:LED_0603_1608Metric, F.Cu at (222.5, 138.5)
- added D27: LED, LED_SMD:LED_0603_1608Metric, F.Cu at (226.6, 117.8)
- added D28: LED, LED_SMD:LED_0603_1608Metric, F.Cu at (226.6, 120.4)
- added D29: LED, LED_SMD:LED_0603_1608Metric, F.Cu at (226.6, 123.0)
- added D30: LED, LED_SMD:LED_0603_1608Metric, F.Cu at (226.6, 125.5)
- added D31: LED, LED_SMD:LED_0603_1608Metric, F.Cu at (226.6, 128.1)
- added D32: LED, LED_SMD:LED_0603_1608Metric, F.Cu at (226.6, 130.7)
- added D33: LED, LED_SMD:LED_0603_1608Metric, F.Cu at (226.6, 133.3)
- added D34: LED, LED_SMD:LED_0603_1608Metric, F.Cu at (226.6, 135.9)
- added D35: LED, LED_SMD:LED_0603_1608Metric, F.Cu at (226.6, 138.5)
- added D36: LED, LED_SMD:LED_0603_1608Metric, F.Cu at (230.6, 117.8)
- added D37: LED, LED_SMD:LED_0603_1608Metric, F.Cu at (230.6, 120.4)
- added D38: LED, LED_SMD:LED_0603_1608Metric, F.Cu at (230.6, 123.0)
- added D39: LED, LED_SMD:LED_0603_1608Metric, F.Cu at (230.6, 125.5)
- added D40: LED, LED_SMD:LED_0603_1608Metric, F.Cu at (230.6, 128.1)
- added D41: LED, LED_SMD:LED_0603_1608Metric, F.Cu at (230.6, 130.7)
- added D42: LED, LED_SMD:LED_0603_1608Metric, F.Cu at (230.6, 133.3)
- added D43: LED, LED_SMD:LED_0603_1608Metric, F.Cu at (230.6, 135.9)
- added D44: LED, LED_SMD:LED_0603_1608Metric, F.Cu at (230.6, 138.5)
- added D45: LED, LED_SMD:LED_0603_1608Metric, F.Cu at (234.7, 117.8)
- added D46: LED, LED_SMD:LED_0603_1608Metric, F.Cu at (234.7, 120.4)
- added D47: LED, LED_SMD:LED_0603_1608Metric, F.Cu at (234.7, 123.0)
- added D48: LED, LED_SMD:LED_0603_1608Metric, F.Cu at (234.7, 125.5)
- added D49: LED, LED_SMD:LED_0603_1608Metric, F.Cu at (234.7, 128.1)
- added J2: Conn_01x02_Socket, Connector_PinSocket_2.54mm:PinSocket_1x02_P2.54mm_Vertical, F.Cu at (184.9, 63.3)
- added Q10: Q_Photo_NPN, LED_SMD:LED_0603_1608Metric, F.Cu at (197.6, 95.0)
- added Q11: Q_Photo_NPN, LED_SMD:LED_0603_1608Metric, F.Cu at (197.6, 100.5)
- added Q12: Q_Photo_NPN, LED_SMD:LED_0603_1608Metric, F.Cu at (197.6, 105.9)
- added Q13: Q_Photo_NPN, LED_SMD:LED_0603_1608Metric, F.Cu at (197.6, 111.4)
- added Q14: Q_Photo_NPN, LED_SMD:LED_0603_1608Metric, F.Cu at (197.6, 116.9)
- added Q15: Q_Photo_NPN, LED_SMD:LED_0603_1608Metric, F.Cu at (197.6, 122.3)
- added Q16: Q_Photo_NPN, LED_SMD:LED_0603_1608Metric, F.Cu at (197.6, 127.8)
- added Q17: NMOS, Package_TO_SOT_THT:TO-251-3-1EP_Horizontal_TabDown, F.Cu at (184.3, 50.8)
- added Q3: Q_Photo_NPN, LED_SMD:LED_0603_1608Metric, F.Cu at (191.7, 100.5)
- added Q4: Q_Photo_NPN, LED_SMD:LED_0603_1608Metric, F.Cu at (191.7, 105.9)
- added Q5: Q_Photo_NPN, LED_SMD:LED_0603_1608Metric, F.Cu at (191.7, 111.4)
- added Q6: Q_Photo_NPN, LED_SMD:LED_0603_1608Metric, F.Cu at (191.7, 116.9)
- added Q7: Q_Photo_NPN, LED_SMD:LED_0603_1608Metric, F.Cu at (191.7, 122.3)
- added Q8: Q_Photo_NPN, LED_SMD:LED_0603_1608Metric, F.Cu at (191.7, 127.8)
- added Q9: Q_Photo_NPN, LED_SMD:LED_0603_1608Metric, F.Cu at (197.6, 89.5)
- added R49: R, Resistor_THT:R_Axial_DIN0207_L6.3mm_D2.5mm_P7.62mm_Horizontal, F.Cu at (123.9, 98.2)
- added R50: R, Resistor_THT:R_Axial_DIN0207_L6.3mm_D2.5mm_P7.62mm_Horizontal, F.Cu at (123.9, 102.3)
- added R51: R, Resistor_THT:R_Axial_DIN0207_L6.3mm_D2.5mm_P7.62mm_Horizontal, F.Cu at (123.9, 106.3)
- added R84: R, Resistor_THT:R_Axial_DIN0207_L6.3mm_D2.5mm_P7.62mm_Horizontal, F.Cu at (145.5, 102.3)
- added R85: R, Resistor_THT:R_Axial_DIN0207_L6.3mm_D2.5mm_P7.62mm_Horizontal, F.Cu at (145.5, 106.3)
- added RN1: R_Network04, Resistor_SMD:R_Array_Convex_4x1206, F.Cu at (215.7, 78.2)
- added RN10: R_Network04, Resistor_SMD:R_Array_Convex_4x1206, F.Cu at (53.2, 81.6)
- added RN11: R_Network04, Resistor_SMD:R_Array_Convex_4x1206, F.Cu at (53.2, 85.8)
- added RN12: R_Network04, Resistor_SMD:R_Array_Convex_4x1206, F.Cu at (53.2, 89.9)
- added RN13: R_Network04, Resistor_SMD:R_Array_Convex_4x1206, F.Cu at (53.2, 94.1)
- added RN14: R_Network04, Resistor_SMD:R_Array_Convex_4x1206, F.Cu at (53.2, 98.3)
- added RN15: R_Network04, Resistor_SMD:R_Array_Convex_4x1206, F.Cu at (53.2, 102.4)
- added RN16: R_Network04, Resistor_SMD:R_Array_Convex_4x1206, F.Cu at (53.2, 106.6)
- added RN2: R_Network04, Resistor_SMD:R_Array_Convex_4x1206, F.Cu at (215.7, 82.4)
- added RN3: R_Network04, Resistor_SMD:R_Array_Convex_4x1206, F.Cu at (215.7, 86.5)
- added RN4: R_Network04, Resistor_SMD:R_Array_Convex_4x1206, F.Cu at (215.7, 90.7)
- added RN5: R_Network04, Resistor_SMD:R_Array_Convex_4x1206, F.Cu at (215.7, 94.9)
- added RN6: R_Network04, Resistor_SMD:R_Array_Convex_4x1206, F.Cu at (215.7, 99.1)
- added RN7: R_Network04, Resistor_SMD:R_Array_Convex_4x1206, F.Cu at (215.7, 103.2)
- added RN8: R_Network04, Resistor_SMD:R_Array_Convex_4x1206, F.Cu at (215.7, 107.4)
- added RN9: R_Network04, Resistor_SMD:R_Array_Convex_4x1206, F.Cu at (53.2, 77.4)
- added RV1: R_Potentiometer_Trim, Connector_PinHeader_2.54mm:PinHeader_1x03_P2.54mm_Vertical, F.Cu at (128.4, 110.7)
- added RV2: R_Potentiometer_Trim, Connector_PinHeader_2.54mm:PinHeader_1x03_P2.54mm_Vertical, F.Cu at (133.0, 110.7)
- added RV3: R_Potentiometer_Trim, Connector_PinHeader_2.54mm:PinHeader_1x03_P2.54mm_Vertical, F.Cu at (137.6, 110.7)
- added RV4: R_Potentiometer_Trim, Connector_PinHeader_2.54mm:PinHeader_1x03_P2.54mm_Vertical, F.Cu at (142.2, 110.7)
- added SW2: SW_DPST_x2, Connector_PinSocket_2.54mm:PinSocket_1x03_P2.54mm_Vertical, F.Cu at (197.6, 41.8)
- added U2: LM393, Package_SO:SOIC-8_3.9x4.9mm_P1.27mm, F.Cu at (105.0, 118.3)
- added U3: LM393, Package_SO:SOIC-8_3.9x4.9mm_P1.27mm, F.Cu at (105.0, 124.9)
- added U4: LM393, Package_SO:SOIC-8_3.9x4.9mm_P1.27mm, F.Cu at (113.5, 111.7)
- added U5: LM393, Package_SO:SOIC-8_3.9x4.9mm_P1.27mm, F.Cu at (113.5, 118.3)
- added U6: LM393, Package_SO:SOIC-8_3.9x4.9mm_P1.27mm, F.Cu at (113.5, 124.9)
- added U7: LM393, Package_SO:SOIC-8_3.9x4.9mm_P1.27mm, F.Cu at (121.9, 111.7)
- added U8: LM393, Package_SO:SOIC-8_3.9x4.9mm_P1.27mm, F.Cu at (121.9, 118.3)
- added U9: LM393, Package_SO:SOIC-8_3.9x4.9mm_P1.27mm, F.Cu at (121.9, 124.9)
- J1: value Conn_01x05_Socket -> Conn_01x04_Socket; footprint Connector_JST:JST_XH_B5B-XH-AM_1x05_P2.50mm_Vertical -> Connector_PinSocket_2.54mm:PinSocket_1x04_P2.54mm_Vertical
- Q1, Q2: footprint LED_THT:LED_D3.0mm -> LED_SMD:LED_0603_1608Metric
- U1: footprint Package_DIP:DIP-8_W7.62mm_Socket_LongPads -> Package_SO:SOIC-8_3.9x4.9mm_P1.27mm
- moved J1 77.0 mm to (193.0, 41.8), turned to 0 degrees
- moved Q1 69.0 mm to (191.7, 89.5)
- moved U1 40.1 mm to (105.0, 111.7)
- moved Q2 31.6 mm to (191.7, 95.0), turned to 0 degrees
Connections:
- J1 pad 1: GND -> Net-(J1-Pin_1)
- J1 pad 2: VCC -> Net-(A1-D0/RX)
- J1 pad 3: Net-(J1-Pin_3) -> GND
- J1 pad 4: Net-(J1-Pin_4) -> VCC
- U1 pad 1: Net-(J1-Pin_5) -> Net-(A1-D11)
- U1 pad 2: Net-(Q1-E) -> Net-(U1A--)
- U1 pad 3: Net-(J1-Pin_3) -> Net-(Q13-E)
- U1 pad 4: GND -> (no net)
- U1 pad 5: Net-(J1-Pin_3) -> Net-(Q14-E)
- U1 pad 6: Net-(Q2-E) -> Net-(U1A--)
- U1 pad 7: Net-(J1-Pin_4) -> Net-(A1-D12)
- U1 pad 8: VCC -> (no net)
Routing:
- net VCC: track 72.9 -> 0.00 mm
- net Net-(J1-Pin_3): track 24.2 -> 0.00 mm
- net Net-(J1-Pin_4): track 20.2 -> 0.00 mm
- net Net-(Q2-E): track 16.1 -> 0.00 mm
- net Net-(Q1-E): track 15.0 -> 0.00 mm
- net Net-(J1-Pin_5): track 11.5 -> 0.00 mm
- net Net-(D2-K): track 2.54 -> 0.00 mm
- net Net-(D1-K): track 2.54 -> 0.00 mm
- net GND: vias 24 -> 0
- removed copper zone on B.Cu, net GND
- removed copper zone on F.Cu, net GND
Other:
- board outline removed

Commit message: 外形の図形10.5
Parts:
- moved RN10 303.5 mm to (344.4, 167.3), turned to -90 degrees
- moved RN9 292.9 mm to (338.9, 142.3), turned to -90 degrees
- moved RN11 279.6 mm to (326.9, 143.3), turned to -90 degrees
- moved RN13 268.7 mm to (317.4, 143.3), turned to -90 degrees
- moved RN14 267.4 mm to (318.4, 132.8), turned to -90 degrees
- moved RN15 258.3 mm to (308.7, 140.8), turned to -90 degrees
- moved RN16 253.6 mm to (305.9, 128.8), turned to -90 degrees
- moved RN12 232.5 mm to (279.5, 143.3), turned to -90 degrees
- moved RN1 231.7 mm to (340.2, 273.6), turned to -90 degrees
- moved RN2 225.9 mm to (336.0, 273.6), turned to -90 degrees
- moved C4 224.7 mm to (268.1, 246.4), turned to 180 degrees
- moved R49 221.1 mm to (330.4, 177.3), turned to -90 degrees
- moved RN3 220.2 mm to (331.9, 273.6), turned to -90 degrees
- moved C5 217.4 mm to (268.1, 242.3), turned to 180 degrees
- moved R50 216.6 mm to (322.9, 187.8), turned to -90 degrees
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Other:
- board outline added: 200 x 200 mm
