File: kiCad/LineSensor_Prot3/LineSensor.kicad_pcb (KiCad board)
At the start: 2 copper layers, 100 x 100 mm, 112 parts, among them J1 Conn_01x04_Socket, J2 Conn_01x02_Socket, Q1 Q_Photo_NPN, Q10 Q_Photo_NPN, Q11 Q_Photo_NPN, Q12 Q_Photo_NPN, Q13 Q_Photo_NPN, Q14 Q_Photo_NPN, Q15 Q_Photo_NPN, Q16 Q_Photo_NPN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

Commit message: 電車
Parts:
- moved C10 0.30 mm to (162.7, 139.6), turned to -170 degrees
- turned C11 to -80 degrees
Routing:
- net VCC: track 0.60 -> 439.3 mm, vias 0 -> 18
- net GND: track 0.35 -> 328.2 mm, vias 0 -> 35
- net Net-(Q17-D): track 0.00 -> 33.3 mm
- net Net-(A1-D13): track 0.00 -> 20.0 mm, vias 0 -> 4
- net Net-(D35-K): track 0.00 -> 8.38 mm
- net Net-(D36-K): track 0.00 -> 7.15 mm
- net Net-(Q8-E): track 0.00 -> 6.07 mm
- net Net-(Q4-E): track 0.00 -> 5.94 mm
- net Net-(Q14-E): track 0.00 -> 5.83 mm
- net Net-(Q2-E): track 0.00 -> 5.73 mm
- net Net-(Q12-E): track 0.00 -> 5.38 mm
- net Net-(Q10-E): track 0.00 -> 5.22 mm
- net Net-(Q16-E): track 0.00 -> 4.98 mm, vias 0 -> 2
- net Net-(Q15-E): track 0.00 -> 4.63 mm
- net Net-(D34-K): track 0.00 -> 4.27 mm
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
Commit message: 電車2
Parts:
- moved A1 129.6 mm to (142.0, 81.1)
- moved SW2 83.1 mm to (80.9, 108.3)
- moved RV1 41.4 mm to (68.3, 141.7)
- moved C2 41.4 mm to (86.5, 142.7)
- moved J1 41.4 mm to (57.1, 141.6)
- moved Q17 41.4 mm to (48.5, 150.6)
- moved RV2 41.4 mm to (72.9, 141.7)
- moved RV3 41.4 mm to (77.5, 141.7)
- moved RV4 41.4 mm to (82.1, 141.7)
- moved R51 24.8 mm to (67.3, 112.3)
- moved J2 24.8 mm to (77.1, 124.7)
- moved R50 24.8 mm to (67.3, 108.2)
- moved R84 24.8 mm to (67.3, 116.3)
- moved R85 24.8 mm to (67.3, 120.4)
- moved C3 24.8 mm to (67.8, 124.4)
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Routing:
- net Net-(Q17-D): track 33.3 -> 315.1 mm, vias 0 -> 26
- net Net-(U3A-+): track 0.00 -> 53.6 mm, vias 0 -> 6
- net Net-(U7A-+): track 0.00 -> 44.2 mm
- net Net-(U2A-+): track 0.00 -> 43.2 mm, vias 0 -> 4
- net GND: track 328.2 -> 367.5 mm, vias 35 -> 39
- net Net-(A1-D4): track 0.00 -> 27.2 mm, vias 0 -> 2
- net Net-(A1-D3): track 0.00 -> 26.3 mm, vias 0 -> 4
- net Net-(A1-A1): track 0.00 -> 25.7 mm, vias 0 -> 2
- net Net-(A1-D5): track 0.00 -> 24.1 mm, vias 0 -> 2
- net Net-(A1-A4): track 0.00 -> 21.9 mm, vias 0 -> 2
- net Net-(Q2-E): track 5.73 -> 27.1 mm, vias 0 -> 4
- net Net-(A1-D12): track 0.00 -> 20.9 mm, vias 0 -> 2
- net Net-(Q6-E): track 0.00 -> 19.9 mm, vias 0 -> 2
- net Net-(A1-D7): track 0.00 -> 19.3 mm, vias 0 -> 4
- net Net-(Q1-E): track 3.31 -> 21.6 mm, vias 0 -> 4
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Other:
- outline, holes or cut-outs redrawn

Commit message: prot4作成
Parts:
- moved RV4 137.4 mm to (215.0, 106.8), turned to 90 degrees
- moved C2 95.2 mm to (162.6, 85.5), turned to -90 degrees
- moved J1 85.7 mm to (130.0, 96.5)
- moved R50 81.9 mm to (147.0, 127.0), turned to -90 degrees
- moved R49 72.3 mm to (137.9, 88.6), turned to 90 degrees
- moved R51 70.9 mm to (137.6, 102.9), turned to -90 degrees
- moved C3 63.1 mm to (67.8, 61.3)
- moved A1 0.55 mm to (142.5, 81.1)
Other:
- outline, holes or cut-outs redrawn
