File: kiCad/LineSensor_Prot5/LineSensor.kicad_pcb (KiCad board)
At the start: 2 copper layers, 100 x 100 mm, 113 parts, among them J1 Conn_01x04_Socket, J2 Conn_01x02_Socket, Q1 Q_Photo_NPN, Q10 Q_Photo_NPN, Q11 Q_Photo_NPN, Q12 Q_Photo_NPN, Q13 Q_Photo_NPN, Q14 Q_Photo_NPN, Q15 Q_Photo_NPN, Q16 Q_Photo_NPN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

Commit message: 11.24朝desktop
Parts:
- moved H1 111.4 mm to (187.0, 126.0)
- moved H2 46.2 mm to (113.1, 126.0)
- moved H3 26.0 mm to (113.0, 74.0)
- moved C8 10.3 mm to (137.8, 72.5)
- moved R11 6.43 mm to (120.7, 65.8)
- moved R46 6.14 mm to (120.3, 133.9)
- moved R45 5.65 mm to (107.3, 114.3)
- moved R24 4.08 mm to (117.7, 79.5)
- moved U5 3.71 mm to (122.9, 82.9)
- moved C7 3.71 mm to (121.0, 87.0)
- moved R23 3.71 mm to (128.8, 81.3)
- moved R42 3.70 mm to (123.1, 63.8)
- moved R3 2.29 mm to (109.9, 120.1)
- moved R2 2.29 mm to (122.4, 135.8)
- moved R19 1.89 mm to (183.5, 130.0)
Changed lines of the file:
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@@
 		(tags "LED")
 		(property "Reference" "D34"
-			(at 0 -1.43 135)
+			(at 0.113413 1.414214 135)
 			(layer "F.SilkS")
 			(effects
@@
 	(footprint "Resistor_SMD:R_0603_1608Metric_Pad0.98x0.95mm_HandSolder"
 		(layer "F.Cu")
-		(at 110.87196 122.203199 22.5)
+		(at 109.85696 120.149199 22.5)
 		(descr "Resistor SMD 0603 (1608 Metric), square (rectangular) end terminal, IPC-7351 nominal with elongated pad for handsoldering. (Body size source: IPC-SM-782 page 72, https://www.pcb-3d.com/wordpress/wp-content/uploads/ipc-sm-782a_amendment_1_and_2.pdf), generated with kicad-footprint-generator")
 		(tags "resistor handsolder")
 		(property "Reference" "R3"
-			(at 0.029087 1.568313 22.5)
+			(at -0.090636 -1.497905 22.5)
 			(layer "F.SilkS")
 			(effects
@@
 	(footprint "Capacitor_SMD:C_0603_1608Metric"
 		(layer "F.Cu")
-		(at 127.836 75.353 180)
+		(at 137.775 72.5 180)
 		(descr "Capacitor SMD 0603 (1608 Metric), square (rectangular) end terminal, IPC-7351 nominal, (Body size source: IPC-SM-782 page 76, https://www.pcb-3d.com/wordpress/wp-content/uploads/ipc-sm-782a_amendment_1_and_2.pdf), generated with kicad-footprint-generator")
 		(tags "capacitor")
 		(property "Reference" "C8"
-			(at 2.507375 -0.175691 0)
+			(at 2.636 -0.147 0)
 			(layer "F.SilkS")
 			(effects
@@
 	(footprint "Package_SO:SOIC-8_3.9x4.9mm_P1.27mm"
 		(layer "F.Cu")
-		(at 120.14 80.428)
+		(at 122.9 82.9)
 		(descr "SOIC, 8 Pin (JEDEC MS-012AA, https://www.analog.com/media/en/package-pcb-resources/package/pkg_pdf/soic_narrow-r/r_8.pdf), generated with kicad-footprint-generator ipc_gullwing_generator.py")
 		(tags "SOIC SO")
@@
 	(footprint "Resistor_SMD:R_0603_1608Metric_Pad0.98x0.95mm_HandSolder"
 		(layer "F.Cu")
-		(at 115.872765 129.646235 -135)
+		(at 120.254765 133.945235 -135)
 		(descr "Resistor SMD 0603 (1608 Metric), square (rectangular) end terminal, IPC-7351 nominal with elongated pad for handsoldering. (Body size source: IPC-SM-782 page 72, https://www.pcb-3d.com/wordpress/wp-content/uploads/ipc-sm-782a_amendment_1_and_2.pdf), generated with kicad-footprint-generator")
 		(tags "resistor handsolder")
 		(property "Reference" "R46"
-			(at 0.634837 1.577017 45)
+			(at 0.077449 -1.414214 45)
 			(layer "F.SilkS")
 			(effects
@@
 	(footprint "Resistor_SMD:R_0603_1608Metric_Pad0.98x0.95mm_HandSolder"
 		(layer "F.Cu")
-		(at 120.605 134.395 50)
+		(at 122.413456 135.799016 50)
 		(descr "Resistor SMD 0603 (1608 Metric), square (rectangular) end terminal, IPC-7351 nominal with elongated pad for handsoldering. (Body size source: IPC-SM-782 page 72, https://www.pcb-3d.com/wordpress/wp-content/uploads/ipc-sm-782a_amendment_1_and_2.pdf), generated with kicad-footprint-generator")
 		(tags "resistor handsolder")
@@
 	(footprint "MountingHole:MountingHole_3.2mm_M3"
 		(layer "F.Cu")
-		(at 110.381 45.167)
+		(at 187 126)
 		(descr "Mounting Hole 3.2mm, M3, no annular, generated by kicad-footprint-generator mountinghole.py")
 		(tags "mountinghole M3")
@@
 	(footprint "Resistor_SMD:R_0603_1608Metric_Pad0.98x0.95mm_HandSolder"
 		(layer "F.Cu")
-		(at 120.311765 66.230765 135)
+		(at 123.054765 63.754765 135)
 		(descr "Resistor SMD 0603 (1608 Metric), square (rectangular) end terminal, IPC-7351 nominal with elongated pad for handsoldering. (Body size source: IPC-SM-782 page 72, https://www.pcb-3d.com/wordpress/wp-content/uploads/ipc-sm-782a_amendment_1_and_2.pdf), generated with kicad-footprint-generator")
 		(tags "resistor handsolder")
@@
 	(footprint "Resistor_SMD:R_0603_1608Metric_Pad0.98x0.95mm_HandSolder"
 		(layer "F.Cu")
-		(at 126.040199 78.82596 -90)
+		(at 128.800199 81.29796 -90)
 		(descr "Resistor SMD 0603 (1608 Metric), square (rectangular) end terminal, IPC-7351 nominal with elongated pad for handsoldering. (Body size source: IPC-SM-782 page 72, https://www.pcb-3d.com/wordpress/wp-content/uploads/ipc-sm-782a_amendment_1_and_2.pdf), generated with kicad-footprint-generator")
 		(tags "resistor handsolder")
@@
 	(footprint "Resistor_SMD:R_0603_1608Metric_Pad0.98x0.95mm_HandSolder"
 		(layer "F.Cu")
-		(at 116.144765 70.333765 -45)
+		(at 120.654765 65.754765 -45)
 		(descr "Resistor SMD 0603 (1608 Metric), square (rectangular) end terminal, IPC-7351 nominal with elongated pad for handsoldering. (Body size source: IPC-SM-782 page 72, https://www.pcb-3d.com/wordpress/wp-content/uploads/ipc-sm-782a_amendment_1_and_2.pdf), generated with kicad-footprint-generator")
 		(tags "resistor handsolder")
@@
 	(footprint "Resistor_SMD:R_0603_1608Metric_Pad0.98x0.95mm_HandSolder"
 		(layer "F.Cu")
-		(at 185.1 129 140)
+		(at 183.500984 130.013456 140)
 		(descr "Resistor SMD 0603 (1608 Metric), square (rectangular) end terminal, IPC-7351 nominal with elongated pad for handsoldering. (Body size source: IPC-SM-782 page 72, https://www.pcb-3d.com/wordpress/wp-content/uploads/ipc-sm-782a_amendment_1_and_2.pdf), generated with kicad-footprint-generator")
 		(tags "resistor handsolder")
@@
 	(footprint "Resistor_SMD:R_0603_1608Metric_Pad0.98x0.95mm_HandSolder"
 		(layer "F.Cu")
-		(at 109.75896 119.412198 -157.5)
+		(at 107.25696 114.349199 -157.5)
 		(descr "Resistor SMD 0603 (1608 Metric), square (rectangular) end terminal, IPC-7351 nominal with elongated pad for handsoldering. (Body size source: IPC-SM-782 page 72, https://www.pcb-3d.com/wordpress/wp-content/uploads/ipc-sm-782a_amendment_1_and_2.pdf), generated with kicad-footprint-generator")
 		(tags "resistor handsolder")
 		(property "Reference" "R45"
-			(at -0.000001 -1.430001 22.5)
+			(at 0.128904 1.405517 22.5)
 			(layer "F.SilkS")
 			(effects
@@
 	(footprint "Capacitor_SMD:C_0603_1608Metric"
 		(layer "F.Cu")
-		(at 118.229936 84.480204 180)
+		(at 120.989936 86.952204 180)
 		(descr "Capacitor SMD 0603 (1608 Metric), square (rectangular) end terminal, IPC-7351 nominal, (Body size source: IPC-SM-782 page 76, https://www.pcb-3d.com/wordpress/wp-content/uploads/ipc-sm-782a_amendment_1_and_2.pdf), generated with kicad-footprint-generator")
 		(tags "capacitor")
@@
 		(tags "LED")
 		(property "Reference" "D42"
-			(at 0.000276 -1.533008 45)
+			(at -0.028008 -1.414214 45)
 			(layer "F.SilkS")
 			(effects
@@
 	(footprint "Resistor_SMD:R_0603_1608Metric_Pad0.98x0.95mm_HandSolder"
 		(layer "F.Cu")
-		(at 114.325765 77.200235 -90)
+		(at 117.7 79.4875 -90)
 		(descr "Resistor SMD 0603 (1608 Metric), square (rectangular) end terminal, IPC-7351 nominal with elongated pad for handsoldering. (Body size source: IPC-SM-782 page 72, https://www.pcb-3d.com/wordpress/wp-content/uploads/ipc-sm-782a_amendment_1_and_2.pdf), generated with kicad-footprint-generator")
 		(tags "resistor handsolder")
 		(property "Reference" "R24"
-			(at 0.000001 -1.43 90)
+			(at 0.1125 1.7 90)
 			(layer "F.SilkS")
 			(effects
@@
 		)
 		(fp_text user "${REFERENCE}"
-			(at 0 0 90)
+			(at 2.472 -2.76 90)
 			(layer "F.Fab")
 			(effects
@@
 	(footprint "MountingHole:MountingHole_3.2mm_M3"
 		(layer "F.Cu")
-		(at 138.887 164.357)
+		(at 113.126 126)
 		(descr "Mounting Hole 3.2mm, M3, no annular, generated by kicad-footprint-generator mountinghole.py")
 		(tags "mountinghole M3")
 		(property "Reference" "H2"
-			(at 32.185 -30.505 90)
+			(at -0.2 -4.8 180)
 			(layer "F.SilkS")
 			(effects
@@
 	(footprint "MountingHole:MountingHole_3.2mm_M3"
 		(layer "F.Cu")
-		(at 113 100)
+		(at 113 74)
 		(descr "Mounting Hole 3.2mm, M3, no annular, generated by kicad-footprint-generator mountinghole.py")
 		(tags "mountinghole M3")
@@
 		(tags "resistor handsolder")
 		(property "Reference" "R43"
-			(at 0 -1.43 157.5)
+			(at -0.064884 1.249112 157.5)
 			(layer "F.SilkS")
 			(effects

Commit message: 11.24桑子チェック1
Parts:
- moved R85 39.9 mm to (171.0, 114.6), turned to 180 degrees
- moved Q17 38.7 mm to (164.5, 119.2), turned to 0 degrees
- moved R84 24.6 mm to (163.4, 110.5), turned to 0 degrees
- moved R16 17.3 mm to (179.5, 65.9), turned to -135 degrees
- moved R15 14.9 mm to (164.4, 57.7), turned to -112.5 degrees
- moved R28 13.6 mm to (186.2, 89.4), turned to 180 degrees
- moved R27 13.3 mm to (193.6, 93.2)
- moved U7 11.5 mm to (187.7, 94.1)
- moved C11 11.4 mm to (186.5, 99.2)
- moved R22 10.0 mm to (140.6, 56.9), turned to 0 degrees
- moved C8 7.86 mm to (142.5, 66.2)
- moved U6 7.86 mm to (144.0, 61.8)
- moved R21 7.71 mm to (150.2, 60.0)
- moved R10 6.32 mm to (129.8, 59.7)
- moved R41 5.94 mm to (135.4, 57.0), turned to -67.5 degrees
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Connections:
- A1 pad 11: U9A -> U9B
- A1 pad 12: U9B -> U9A
- A1 pad 14: U3B -> U3A
- A1 pad 15: U3A -> U3B
- A1 pad 19: U3B -> U4B
- A1 pad 20: U3A -> U4A
- A1 pad 23: U6B -> U6A
- A1 pad 24: U6A -> U6B
- R15 pad 1: Net-(Q7-E) -> Net-(Q8-E)
- R16 pad 1: Net-(Q8-E) -> Net-(Q7-E)
- U8 pad 2: Net-(Q7-E) -> Net-(Q8-E)
- U8 pad 6: Net-(Q8-E) -> Net-(Q7-E)
Routing:
- net VCC: track 0.00 -> 663.7 mm, vias 0 -> 36
- net GND: track 0.00 -> 490.1 mm, vias 0 -> 24
- net Net-(U2A-+): track 0.00 -> 294.8 mm, vias 0 -> 14
- net U6B: track 0.00 -> 48.6 mm, vias 0 -> 3
- net U2B: track 0.00 -> 47.1 mm, vias 0 -> 1
- net U5A: track 0.00 -> 46.4 mm, vias 0 -> 2
- net U3B: track 0.00 -> 46.4 mm, vias 0 -> 1
- net U6A: track 0.00 -> 46.3 mm, vias 0 -> 1
- net U8A: track 0.00 -> 41.9 mm, vias 0 -> 2
- net U8B: track 0.00 -> 41.1 mm, vias 0 -> 2
- net U7B: track 0.00 -> 39.4 mm
- net U3A: track 0.00 -> 38.0 mm, vias 0 -> 1
- net U9B: track 0.00 -> 36.8 mm, vias 0 -> 1
- net U5B: track 0.00 -> 36.6 mm, vias 0 -> 1
- net U2A: track 0.00 -> 34.2 mm, vias 0 -> 1
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
Commit message: 完成？(GPIO照らし合わせ)
Parts:
- moved C7 0.89 mm to (120.4, 87.6), turned to 90 degrees
Routing:
- net Net-(Q17-D): track 27.0 -> 372.9 mm, vias 2 -> 24
- net GND: track 490.1 -> 633.8 mm
- net VCC: track 663.7 -> 698.1 mm, vias 36 -> 37
- net Net-(Q5-E): track 3.30 -> 19.5 mm, vias 0 -> 2
- net Net-(Q14-E): track 5.38 -> 18.1 mm, vias 0 -> 2
- net Net-(A1-D1/TX): track 0.00 -> 4.14 mm
- net Net-(D36-K): track 0.29 -> 3.85 mm
- net U5A: vias 2 -> 1
Other:
- board text added: "11"
- board text added: "12"
- board text added: "2"
- board text added: "3"
- board text added: "4"
- board text added: "5"
- board text added: "6"
- board text added: "7"
- board text added: "8"
- board text added: "9"
- board text added: "A0"
- board text added: "A1"
- board text added: "A2"
- board text added: "A3"
- board text added: "A4"
- board text added: "A5"

Commit message: 11.25チーム名印字など
Other:
- board text added: "2025"
- board text added: "URAWA BOLSAE"

Commit message: ガーバー作成1
Parts:
- J2: footprint Connector_PinSocket_2.54mm:PinSocket_1x02_P2.54mm_Vertical -> Connector_JST:JST_XH_B2B-XH-A_1x02_P2.50mm_Vertical
- moved R50 0.93 mm to (176.8, 109.8)
- moved J2 0.85 mm to (168.9, 105.4), turned to 0 degrees
Routing:
- net Net-(R50-Pad1): track 4.79 -> 3.91 mm
