File: kiCad/LineSensor_Prot5/LineSensor.kicad_sch (KiCad schematic)
At the start: 113 parts, among them J1 Conn_01x04_Socket, J2 Conn_01x02_Socket, Q1 Q_Photo_NPN, Q10 Q_Photo_NPN, Q11 Q_Photo_NPN, Q12 Q_Photo_NPN, Q13 Q_Photo_NPN, Q14 Q_Photo_NPN, Q15 Q_Photo_NPN, Q16 Q_Photo_NPN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

Commit message: 11.24桑子チェック1
Connections:
- net U3A: now also A1.14 (D11); no longer A1.15 (D12), A1.20 (A1)
- net U3B: now also A1.15 (D12); no longer A1.14 (D11), A1.19 (A0)
- net U4A: now also A1.20 (A1)
- net U4B: now also A1.19 (A0)
- net U6A: now also A1.23 (A4); no longer A1.24 (A5)
- net U6B: now also A1.24 (A5); no longer A1.23 (A4)
- net U9A: now also A1.12 (D9); no longer A1.11 (D8)
- net U9B: now also A1.11 (D8); no longer A1.12 (D9)
- net at R15.1, U8.2 (-): now also Q8.2 (E); no longer Q7.2 (E)
- net at R16.1, U8.6 (-): now also Q7.2 (E); no longer Q8.2 (E)
Other:
- moved on the sheet: Q7, Q8
Changed lines of the file:
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@@
 	)
 	(junction
+		(at 693.42 495.3)
+		(diameter 0)
+		(color 0 0 0 0)
+	)
+	(junction
 		(at 312.42 546.1)
 		(diameter 0)
@@
 	)
 	(junction
-		(at 693.42 495.3)
-		(diameter 0)
-		(color 0 0 0 0)
-	)
-	(junction
 		(at 535.94 561.34)
 		(diameter 0)
@@
 	)
 	(junction
-		(at 673.1 495.3)
-		(diameter 0)
-		(color 0 0 0 0)
-	)
-	(junction
 		(at 431.8 486.41)
 		(diameter 0)
@@
 	)
 	(junction
+		(at 673.1 495.3)
+		(diameter 0)
+		(color 0 0 0 0)
+	)
+	(junction
 		(at 509.27 541.02)
 		(diameter 0)
@@
 	)
 	(junction
-		(at 693.42 505.46)
-		(diameter 0)
-		(color 0 0 0 0)
-	)
-	(junction
 		(at 350.52 546.1)
 		(diameter 0)
@@
 	)
 	(junction
+		(at 693.42 505.46)
+		(diameter 0)
+		(color 0 0 0 0)
+	)
+	(junction
 		(at 350.52 562.61)
 		(diameter 0)
@@
 	(wire
 		(pts
-			(xy 693.42 505.46) (xy 713.74 505.46)
+			(xy 673.1 505.46) (xy 693.42 505.46)
 		)
 		(stroke
@@
 	(wire
 		(pts
-			(xy 673.1 505.46) (xy 693.42 505.46)
-		)
-		(stroke
-			(width 0)
-			(type default)
-		)
-	)
-	(wire
-		(pts
 			(xy 189.23 412.75) (xy 189.23 415.29)
 		)
@@
 	(wire
 		(pts
+			(xy 693.42 505.46) (xy 713.74 505.46)
+		)
+		(stroke
+			(width 0)
+			(type default)
+		)
+	)
+	(wire
+		(pts
 			(xy 359.41 562.61) (xy 369.57 562.61)
 		)
@@
 	(global_label "U9A"
 		(shape bidirectional)
-		(at 541.02 427.99 180)
+		(at 541.02 430.53 180)
 		(fields_autoplaced yes)
 		(effects
@@
 		)
 		(property "Intersheetrefs" "${INTERSHEET_REFS}"
-			(at 533.2949 427.99 0)
+			(at 533.2949 430.53 0)
 			(effects
 				(font
@@
 		)
 	)
-	(global_label "U3A"
+	(global_label "U4A"
 		(shape bidirectional)
-		(at 541.02 438.15 180)
+		(at 566.42 425.45 0)
 		(fields_autoplaced yes)
 		(effects
@@
 				(size 1.27 1.27)
 			)
-			(justify right)
+			(justify left)
 		)
 		(property "Intersheetrefs" "${INTERSHEET_REFS}"
-			(at 533.2949 438.15 0)
+			(at 574.1451 425.45 0)
 			(effects
 				(font
 					(size 1.27 1.27)
 				)
-				(justify right)
+				(justify left)
 				(hide yes)
 			)
@@
 	(global_label "U6B"
 		(shape bidirectional)
-		(at 566.42 433.07 0)
+		(at 566.42 435.61 0)
 		(fields_autoplaced yes)
 		(effects
@@
 		)
 		(property "Intersheetrefs" "${INTERSHEET_REFS}"
-			(at 574.3265 433.07 0)
+			(at 574.3265 435.61 0)
 			(effects
 				(font
@@
 	(global_label "U6A"
 		(shape bidirectional)
-		(at 566.42 435.61 0)
+		(at 566.42 433.07 0)
 		(fields_autoplaced yes)
 		(effects
@@
 		)
 		(property "Intersheetrefs" "${INTERSHEET_REFS}"
-			(at 574.1451 435.61 0)
+			(at 574.1451 433.07 0)
 			(effects
 				(font
@@
 		)
 	)
-	(global_label "U3B"
+	(global_label "U4B"
 		(shape bidirectional)
-		(at 541.02 435.61 180)
+		(at 566.42 422.91 0)
 		(fields_autoplaced yes)
 		(effects
@@
 				(size 1.27 1.27)
 			)
-			(justify right)
+			(justify left)
 		)
 		(property "Intersheetrefs" "${INTERSHEET_REFS}"
-			(at 533.1135 435.61 0)
+			(at 574.3265 422.91 0)
 			(effects
 				(font
 					(size 1.27 1.27)
 				)
-				(justify right)
+				(justify left)
 				(hide yes)
 			)
@@
 	(global_label "U9B"
 		(shape bidirectional)
-		(at 541.02 430.53 180)
+		(at 541.02 427.99 180)
 		(fields_autoplaced yes)
 		(effects
@@
 		)
 		(property "Intersheetrefs" "${INTERSHEET_REFS}"
-			(at 533.1135 430.53 0)
+			(at 533.1135 427.99 0)
 			(effects
 				(font
@@
 	(global_label "U3A"
 		(shape bidirectional)
-		(at 566.42 425.45 0)
+		(at 541.02 435.61 180)
 		(fields_autoplaced yes)
 		(effects
@@
 				(size 1.27 1.27)
 			)
-			(justify left)
+			(justify right)
 		)
 		(property "Intersheetrefs" "${INTERSHEET_REFS}"
-			(at 574.1451 425.45 0)
+			(at 533.2949 435.61 0)
 			(effects
 				(font
 					(size 1.27 1.27)
 				)
-				(justify left)
+				(justify right)
 				(hide yes)
 			)
@@
 	(global_label "U3B"
 		(shape bidirectional)
-		(at 566.42 422.91 0)
+		(at 541.02 438.15 180)
 		(fields_autoplaced yes)
 		(effects
@@
 				(size 1.27 1.27)
 			)
-			(justify left)
+			(justify right)
 		)
 		(property "Intersheetrefs" "${INTERSHEET_REFS}"
-			(at 574.3265 422.91 0)
+			(at 533.1135 438.15 0)
 			(effects
 				(font
 					(size 1.27 1.27)
 				)
-				(justify left)
+				(justify right)
 				(hide yes)
 			)
@@
 	(symbol
 		(lib_id "Device:Q_Photo_NPN")
-		(at 690.88 500.38 0)
+		(at 670.56 500.38 0)
 		(mirror x)
 		(unit 1)
@@
 		(fields_autoplaced yes)
 		(property "Reference" "Q7"
-			(at 695.96 502.3994 0)
+			(at 675.64 502.3994 0)
 			(effects
 				(font
@@
 		)
 		(property "Value" "Q_Photo_NPN"
-			(at 695.96 499.8594 0)
+			(at 675.64 499.8594 0)
 			(effects
 				(font
@@
 		)
 		(property "Footprint" "NJL7502R:NJL7502R"
-			(at 695.96 502.92 0)
+			(at 675.64 502.92 0)
 			(effects
 				(font
@@
 		)
 		(property "Datasheet" "~"
-			(at 690.88 500.38 0)
+			(at 670.56 500.38 0)
 			(effects
 				(font
@@
 		)
 		(property "Description" "NPN phototransistor, collector/emitter"
-			(at 690.88 500.38 0)
+			(at 670.56 500.38 0)
 			(effects
 				(font
@@
 	(symbol
 		(lib_id "Device:Q_Photo_NPN")
-		(at 670.56 500.38 0)
+		(at 690.88 500.38 0)
 		(mirror x)
 		(unit 1)
@@
 		(fields_autoplaced yes)
 		(property "Reference" "Q8"
-			(at 675.64 502.3994 0)
+			(at 695.96 502.3994 0)
 			(effects
 				(font
@@
 		)
 		(property "Value" "Q_Photo_NPN"
-			(at 675.64 499.8594 0)
+			(at 695.96 499.8594 0)
 			(effects
 				(font
@@
 		)
 		(property "Footprint" "NJL7502R:NJL7502R"
-			(at 675.64 502.92 0)
+			(at 695.96 502.92 0)
 			(effects
 				(font
@@
 		)
 		(property "Datasheet" "~"
-			(at 670.56 500.38 0)
+			(at 690.88 500.38 0)
 			(effects
 				(font
@@
 		)
 		(property "Description" "NPN phototransistor, collector/emitter"
-			(at 670.56 500.38 0)
+			(at 690.88 500.38 0)
 			(effects
 				(font

Commit message: 完成？(GPIO照らし合わせ)
Connections:
- no-connect marks 0 -> 1
Changed lines of the file:
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@@
 		(color 0 0 0 0)
+	)
+	(no_connect
+		(at 450.85 325.12)
 	)
 	(wire

Commit message: ガーバー作成1
Parts:
- J2: footprint Connector_PinSocket_2.54mm:PinSocket_1x02_P2.54mm_Vertical -> Connector_JST:JST_XH_B2B-XH-A_1x02_P2.50mm_Vertical
Changed lines of the file:
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@@
 			)
 		)
-		(property "Footprint" "Connector_PinSocket_2.54mm:PinSocket_1x02_P2.54mm_Vertical"
+		(property "Footprint" "Connector_JST:JST_XH_B2B-XH-A_1x02_P2.50mm_Vertical"
 			(at 601.98 186.69 0)
 			(effects
