File: kiCad/TBTMOTOR/TB67H450FNGｘ４/TB67H450FNGｘ４.kicad_pcb (KiCad board)
At the start: 2 copper layers, 19 parts, among them J1 Conn_01x02_Socket, J2 Conn_01x02_Socket, J3 Conn_01x02_Socket, J4 Conn_01x02_Socket, J5 Conn_01x02_Socket, J6 Conn_01x10_Socket, SW1 SW_DPST_x2

Commit message: EEPROM試験完了
Parts:
- J1, J2, J3, J4: footprint Connector_AMASS:AMASS_XT30U-M_1x02_P5.0mm_Vertical -> Connector_JST:JST_XH_B2B-XH-A_1x02_P2.50mm_Vertical
- moved C4 83.6 mm to (174.2, 45.2)
- moved C3 78.2 mm to (178.8, 40.9), turned to 90 degrees
- moved U2 75.7 mm to (171.0, 33.6), turned to 90 degrees
- moved U4 73.5 mm to (169.5, 55.5), turned to 90 degrees
- moved U3 73.0 mm to (186.4, 35.0), turned to -90 degrees
- moved C2 68.0 mm to (183.1, 45.0), turned to 0 degrees
- moved C1 62.1 mm to (178.6, 49.3), turned to -90 degrees
- moved SW1 49.9 mm to (152.9, 72.0)
- moved U1 47.7 mm to (186.3, 55.1), turned to -90 degrees
- moved J4 4.45 mm to (225.7, 88.5), turned to 0 degrees
- moved J3 2.67 mm to (212.7, 88.5), turned to 0 degrees
- moved J1 2.05 mm to (186.6, 89.0), turned to 0 degrees
- moved R4 1.59 mm to (233.1, 96.4)
- moved J2 0.60 mm to (199.7, 88.8), turned to 0 degrees
Connections:
- R2 pad 1: Net-(U1-RS) -> Net-(U2-RS)
- R3 pad 2: Net-(U1-RS) -> Net-(U3-RS)
- R4 pad 1: Net-(U1-RS) -> Net-(U4-RS)
- U2 pad 7: Net-(U1-RS) -> Net-(U2-RS)
- U3 pad 7: Net-(U1-RS) -> Net-(U3-RS)
- U4 pad 7: Net-(U1-RS) -> Net-(U4-RS)
Other:
- board outline added: 75.7 x 98.9 mm
