File: kiCad/TBTMOTOR/TB67H450FNGｘ４/TB67H450FNGｘ４.kicad_sch (KiCad schematic)
At the start: 19 parts, among them J1 Conn_01x02_Socket, J2 Conn_01x02_Socket, J3 Conn_01x02_Socket, J4 Conn_01x02_Socket, J5 Conn_01x02_Socket, J6 Conn_01x10_Socket, SW1 SW_DPST_x2

Commit message: EEPROM試験完了
Parts:
- added H1, H2, H3, H4: MountingHole, symbol Mechanical:MountingHole
- J1, J2, J3, J4: footprint Connector_AMASS:AMASS_XT30U-M_1x02_P5.0mm_Vertical -> Connector_JST:JST_XH_B2B-XH-A_1x02_P2.50mm_Vertical
Connections:
- net VERF is gone; now on net VREF: J6.1 (Pin_1), U3.4 (VREF), U4.4 (VREF)
- new net: R4.1, U4.7 (RS)
- new net: R3.2, U3.7 (RS)
- new net: R1.1, U1.7 (RS)
- new net: R2.1, U2.7 (RS)
Other:
- moved on the sheet: R3, R4
