File: kiCad/LineSensor_Block_prot1/LineSensor_Block_prot1.kicad_pcb (KiCad board)
At the start: 2 copper layers, 46 parts, among them J1 Conn_01x07_Socket, J2 Conn_01x07_Socket, Q1 Q_Photo_NPN, Q10 Q_Photo_NPN, Q11 Q_Photo_NPN, Q12 Q_Photo_NPN, Q13 Q_Photo_NPN, Q14 Q_Photo_NPN, Q15 Q_Photo_NPN, Q16 Q_Photo_NPN, Q2 Q_Photo_NPN, Q3 Q_Photo_NPN, Q4 Q_Photo_NPN, Q5 Q_Photo_NPN, Q6 Q_Photo_NPN, Q7 Q_Photo_NPN, Q8 Q_Photo_NPN, Q9 Q_Photo_NPN

Commit message: ラインセンサー外側の配置と配線
Parts:
- removed D15, D16: LED, LED_SMD:LED_0603_1608Metric
- removed the D7 at (58.6, 108.0)
- removed the D8 at (58.6, 110.6)
- removed Q15: Q_Photo_NPN, LED_SMD:LED_0603_1608Metric
- removed Q16: Q_Photo_NPN, Capacitor_SMD:C_0603_1608Metric
- removed the Q7 at (66.7, 108.0)
- removed the Q8 at (66.7, 110.6)
- removed RN1, RN2, RN3, RN4, RN5, RN6, RN7, RN8: R_Network04, Resistor_SMD:R_Array_Convex_4x1206
- removed U3: ~, Package_SO:TSSOP-16_4.4x5mm_P0.65mm
- added C10: C, Capacitor_SMD:C_0603_1608Metric, F.Cu at (74.8, 57.1)
- added C11: C, Capacitor_SMD:C_0603_1608Metric, F.Cu at (74.8, 59.6)
- added C12: C, Capacitor_SMD:C_0603_1608Metric, F.Cu at (74.8, 62.2)
- added C13: C, Capacitor_SMD:C_0603_1608Metric, F.Cu at (530.0, -49.0)
- added C14: C, Capacitor_SMD:C_0603_1608Metric, F.Cu at (32.6, 107.9)
- added C3: C, Capacitor_SMD:C_0603_1608Metric, F.Cu at (559.8, -30.3)
- added C4: C, Capacitor_SMD:C_0603_1608Metric, F.Cu at (550.4, -43.8)
- added C5: C, Capacitor_SMD:C_0603_1608Metric, F.Cu at (536.4, -56.1)
- added C6: C, Capacitor_SMD:C_0603_1608Metric, F.Cu at (521.1, -63.9)
- added C7: C, Resistor_SMD:R_0603_1608Metric, F.Cu at (70.8, 72.2)
- added C8: C, Capacitor_SMD:C_0603_1608Metric, F.Cu at (74.8, 52.1)
- added C9: C, Capacitor_SMD:C_0603_1608Metric, F.Cu at (74.8, 54.6)
- added H1: MountingHole, MountingHole:MountingHole_3.2mm_M3, F.Cu at (559.6, -7.31)
- added H2: MountingHole, MountingHole:MountingHole_3.2mm_M3, F.Cu at (523.4, -55.2)
- added H3: MountingHole, MountingHole:MountingHole_3.2mm_M3, F.Cu at (419.1, -34.1)
- added H4: MountingHole, MountingHole:MountingHole_3.2mm_M3, F.Cu at (419.1, -26.1)
- added J3: Conn_01x07_Socket, Pinsocket_and_pinheader:PinSocket_1x07_P2.54mm_Horizontal_edited, B.Cu at (482.2, 14.9)
- added J4: Conn_01x07_Socket, Pinsocket_and_pinheader:PinSocket_1x07_P2.54mm_Horizontal_edited, B.Cu at (471.1, -22.6)
- added R1: R, Resistor_SMD:R_0603_1608Metric, F.Cu at (567.1, 6.30)
- added R10: R, Resistor_SMD:R_0603_1608Metric, F.Cu at (79.2, 76.2)
- added R10d1: R, Resistor_SMD:R_0603_1608Metric, F.Cu at (84.3, 120.5)
- added R11: R, Resistor_SMD:R_0603_1608Metric, F.Cu at (82.8, 54.6)
- added R11d1: R, Resistor_SMD:R_0603_1608Metric, F.Cu at (84.2, 123.1)
- added R12: R, Resistor_SMD:R_0603_1608Metric, F.Cu at (82.8, 57.1)
- added R12d1: R, Resistor_SMD:R_0603_1608Metric, F.Cu at (84.2, 125.7)
- added R1d1: R, Resistor_SMD:R_0603_1608Metric, F.Cu at (562.0, 0.00)
- added R2: R, Resistor_SMD:R_0603_1608Metric, F.Cu at (566.4, -11.0)
- added R2d1: R, Resistor_SMD:R_0603_1608Metric, F.Cu at (559.9, -16.0)
- added R3: R, Resistor_SMD:R_0603_1608Metric, F.Cu at (561.2, -27.7)
- added R3d1: R, Resistor_SMD:R_0603_1608Metric, F.Cu at (553.7, -31.0)
- added R4: R, Resistor_SMD:R_0603_1608Metric, F.Cu at (552.3, -41.7)
- added R4d1: R, Resistor_SMD:R_0603_1608Metric, F.Cu at (543.8, -43.8)
- added R5: R, Resistor_SMD:R_0603_1608Metric, F.Cu at (538.6, -54.3)
- added R5d1: R, Resistor_SMD:R_0603_1608Metric, F.Cu at (531.0, -53.7)
- added R6: R, Resistor_SMD:R_0603_1608Metric, F.Cu at (523.8, -62.5)
- added R6d1: R, Resistor_SMD:R_0603_1608Metric, F.Cu at (516.0, -59.9)
- added R7: R, Resistor_SMD:R_0603_1608Metric, F.Cu at (78.8, 67.2)
- added R7d1: R, Resistor_SMD:R_0603_1608Metric, F.Cu at (68.8, 139.1)
- added R8: R, Resistor_SMD:R_0603_1608Metric, F.Cu at (78.8, 69.7)
- added R8d1: R, Resistor_SMD:R_0603_1608Metric, F.Cu at (52.8, 141.2)
- added R9: R, Resistor_SMD:R_0603_1608Metric, F.Cu at (78.8, 72.2)
- added R9d1: R, Resistor_SMD:R_0603_1608Metric, F.Cu at (88.4, 136.6)
- added U1: ~, Package_SO:TSSOP-16_4.4x5mm_P0.65mm, F.Cu at (537.2, -46.0)
- J1, J2: footprint Connector_JST2:JST_PH_B7B-PH-SM4-TB_1x07-1MP_P2.00mm_Vertical -> Pinsocket_and_pinheader:PinHeader_1x07_P2.54mm_Horizontal_edited; moved to B.Cu
- moved D2 516.4 mm to (562.8, -16.8), turned to 105 degrees
- moved D1 514.8 mm to (565.0, 0.00), turned to 90 degrees
- moved D3 514.4 mm to (556.3, -32.5), turned to 120 degrees
- moved Q2 511.5 mm to (565.7, -17.6), turned to -75 degrees
- moved Q1 509.8 mm to (568.0, 0.00), turned to -90 degrees
- moved Q3 509.5 mm to (558.9, -34.0), turned to -60 degrees
- moved D4 508.8 mm to (546.0, -46.0), turned to 135 degrees
- moved Q4 503.7 mm to (548.1, -48.1), turned to -45 degrees
- moved D5 499.9 mm to (532.5, -56.3), turned to 150 degrees
- moved Q5 494.5 mm to (534.0, -58.9), turned to -30 degrees
- moved C2 493.4 mm to (565.7, -13.8), turned to -165 degrees
- moved C1 490.1 mm to (567.1, 3.35), turned to 180 degrees
- moved D6 488.1 mm to (516.8, -62.8), turned to 165 degrees
- moved Q6 482.3 mm to (517.6, -65.7), turned to -15 degrees
- moved J1 371.5 mm to (512.1, 22.6), turned to -144 degrees
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- renumbered D12 to D10, D13 to D11, D14 to D12, D9 to D7, D10 to D8, D11 to D9, Q12 to Q10, Q13 to Q11, Q14 to Q12, Q9 to Q7, Q10 to Q8, Q11 to Q9
Connections:
- C1 pad 1: GND1 -> Net-(Q1-E)
- C1 pad 2: 3v3_１ -> GND1
- C2 pad 1: GND1 -> Net-(Q2-E)
- C2 pad 2: 3v3_1 -> GND1
- Q10 pad 2: Net-(Q12-E) -> Net-(Q10-E)
- Q11 pad 2: Net-(Q13-E) -> Net-(Q11-E)
- Q12 pad 2: Net-(Q14-E) -> Net-(Q12-E)
- Q7 pad 2: Net-(Q9-E) -> Net-(Q7-E)
- Q8 pad 2: Net-(Q10-E) -> Net-(Q8-E)
- Q9 pad 2: Net-(Q11-E) -> Net-(Q9-E)
- U2 pad 1: Net-(Q4-E) -> Net-(Q10-E)
- U2 pad 10: MUX1B -> MUX2B
- U2 pad 11: MUX1A -> MUX2A
- U2 pad 12: Net-(Q8-E) -> unconnected-(U2-3-Pad12)
- U2 pad 13: Net-(Q7-E) -> unconnected-(U2-0-Pad13)
- U2 pad 14: (no net) -> Net-(Q12-E)
- U2 pad 15: (no net) -> Net-(Q11-E)
- U2 pad 2: Net-(Q3-E) -> Net-(Q9-E)
- U2 pad 3: (no net) -> MUX2COM
- U2 pad 4: (no net) -> Net-(Q8-E)
- U2 pad 5: (no net) -> Net-(Q7-E)
- U2 pad 6: (no net) -> GND1
- U2 pad 7: (no net) -> GND1
- U2 pad 8: (no net) -> GND1
- U2 pad 9: MUX1C -> MUX2C
Routing:
- net 3v3_1: track 0.00 -> 93.2 mm
- net LED_5V_1: track 0.00 -> 89.9 mm
- net GND1: track 0.00 -> 17.7 mm
- net Net-(Q4-E): track 0.00 -> 6.99 mm
- net Net-(Q6-E): track 0.00 -> 6.01 mm
- net Net-(Q3-E): track 0.00 -> 5.88 mm
- net Net-(Q2-E): track 0.00 -> 5.74 mm
- net Net-(Q5-E): track 0.00 -> 5.63 mm
- net Net-(Q1-E): track 0.00 -> 5.56 mm
- net Net-(D4-K): track 0.00 -> 3.02 mm
- net Net-(D1-K): track 0.00 -> 3.02 mm
- net Net-(D6-K): track 0.00 -> 3.00 mm
- net Net-(D2-K): track 0.00 -> 3.00 mm
- net Net-(D3-K): track 0.00 -> 3.00 mm
- net Net-(D5-K): track 0.00 -> 2.98 mm
Other:
- board outline added: 140 x 140 mm

Commit message: マルチプレクソ16chにするくそ
Parts:
- added U4: ~, seeeduino:名称未設定, F.Cu at (399.0, 59.0)
- moved J4 126.2 mm to (371.7, 55.3)
- moved C2 123.0 mm to (462.4, 52.9)
- moved D5 123.0 mm to (429.1, 10.5)
- moved R5 123.0 mm to (435.3, 12.5)
- moved C4 123.0 mm to (447.0, 23.0)
- moved C5 123.0 mm to (433.0, 10.7)
- moved C6 123.0 mm to (417.8, 2.93)
- moved D1 123.0 mm to (461.7, 66.8)
- moved D3 123.0 mm to (453.0, 34.3)
- moved D4 123.0 mm to (442.6, 20.8)
- moved H1 123.0 mm to (456.2, 59.5)
- moved J1 123.0 mm to (408.8, 89.4)
- moved J3 123.0 mm to (378.8, 81.7)
- moved Q1 123.0 mm to (464.7, 66.8)
- moved Q2 123.0 mm to (462.4, 49.2)
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