File: kiCad/LineSensor_Block_prot2/LineSensor_Block_prot2.kicad_pcb (KiCad board)
At the start: 2 copper layers, 336.4 x 337.8 mm, 76 parts, among them J1 Conn_01x08_Socket, J2 Conn_01x08_Socket, J3 Conn_01x08_Socket, J4 Conn_01x08_Socket, J5 Conn_01x08_Socket, J6 Conn_01x08_Socket, J7 Conn_01x03_Socket, Q1 Q_Photo_NPN, Q10 Q_Photo_NPN, Q11 Q_Photo_NPN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

Commit message: 24夜まで
Parts:
- removed C1, C10, C11, C12, C13, C14, C2, C3, C4, C5, C6, C8, C9: C, Capacitor_SMD:C_0603_1608Metric
- removed C7: C, Resistor_SMD:R_0603_1608Metric
- removed J7: Conn_01x03_Socket, Connector_JST:JST_XH_B3B-XH-AM_1x03_P2.50mm_Vertical
Connections:
- Q1 pad 1: 3v3_1 -> Net-(J5-Pin_8)
- Q1 pad 2: Net-(J5-Pin_8) -> GND1
- Q10 pad 1: 3v3_1 -> Net-(J6-Pin_5)
- Q10 pad 2: Net-(J6-Pin_5) -> GND1
- Q11 pad 1: 3v3_1 -> Net-(J6-Pin_4)
- Q11 pad 2: Net-(J6-Pin_4) -> GND1
- Q12 pad 1: 3v3_1 -> Net-(J6-Pin_3)
- Q12 pad 2: Net-(J6-Pin_3) -> GND1
- Q2 pad 1: 3v3_1 -> Net-(J5-Pin_7)
- Q2 pad 2: Net-(J5-Pin_7) -> GND1
- Q3 pad 1: 3v3_1 -> Net-(J5-Pin_6)
- Q3 pad 2: Net-(J5-Pin_6) -> GND1
- Q4 pad 1: 3v3_1 -> Net-(J5-Pin_5)
- Q4 pad 2: Net-(J5-Pin_5) -> GND1
- Q5 pad 1: 3v3_1 -> Net-(J5-Pin_4)
- Q5 pad 2: Net-(J5-Pin_4) -> GND1
- Q6 pad 1: 3v3_1 -> Net-(J5-Pin_3)
- Q6 pad 2: Net-(J5-Pin_3) -> GND1
- Q7 pad 1: 3v3_1 -> Net-(J6-Pin_8)
- Q7 pad 2: Net-(J6-Pin_8) -> GND1
- Q8 pad 1: 3v3_1 -> Net-(J6-Pin_7)
- Q8 pad 2: Net-(J6-Pin_7) -> GND1
- Q9 pad 1: 3v3_1 -> Net-(J6-Pin_6)
- Q9 pad 2: Net-(J6-Pin_6) -> GND1
- R1 pad 1: Net-(J5-Pin_8) -> 3v3_1
- R1 pad 2: GND1 -> Net-(J5-Pin_8)
- R10 pad 1: Net-(J6-Pin_5) -> 3v3_1
- R10 pad 2: GND1 -> Net-(J6-Pin_5)
- R11 pad 1: Net-(J6-Pin_4) -> 3v3_1
- R11 pad 2: GND1 -> Net-(J6-Pin_4)
- R12 pad 1: Net-(J6-Pin_3) -> 3v3_1
- R12 pad 2: GND1 -> Net-(J6-Pin_3)
- R2 pad 1: Net-(J5-Pin_7) -> 3v3_1
- R2 pad 2: GND1 -> Net-(J5-Pin_7)
- R3 pad 1: Net-(J5-Pin_6) -> 3v3_1
- R3 pad 2: GND1 -> Net-(J5-Pin_6)
- R4 pad 1: Net-(J5-Pin_5) -> 3v3_1
- R4 pad 2: GND1 -> Net-(J5-Pin_5)
- R5 pad 1: Net-(J5-Pin_4) -> 3v3_1
- R5 pad 2: GND1 -> Net-(J5-Pin_4)
- R6 pad 1: Net-(J5-Pin_3) -> 3v3_1
- R6 pad 2: GND1 -> Net-(J5-Pin_3)
- R7 pad 1: Net-(J6-Pin_8) -> 3v3_1
- R7 pad 2: GND1 -> Net-(J6-Pin_8)
- R8 pad 1: Net-(J6-Pin_7) -> 3v3_1
- R8 pad 2: GND1 -> Net-(J6-Pin_7)
- R9 pad 1: Net-(J6-Pin_6) -> 3v3_1
- R9 pad 2: GND1 -> Net-(J6-Pin_6)
- U1 pad 15: GND1 -> Net-(U1-~{E})
- U2 pad 10: Net-(U2-S0) -> Net-(U1-S0)
- U2 pad 11: Net-(U2-S1) -> Net-(U1-S1)
- U2 pad 13: Net-(U2-S3) -> Net-(U1-S3)
- U2 pad 14: Net-(U2-S2) -> Net-(U1-S2)
- U2 pad 15: GND1 -> Net-(U2-~{E})
- U4 pad 10: Net-(U2-S1) -> Net-(U1-~{E})
- U4 pad 11: Net-(U2-S0) -> unconnected-(U4-10-Pad11)
- U4 pad 2: Net-(U2-COM) -> Net-(U1-S3)
- U4 pad 3: Net-(U1-S3) -> Net-(U1-S2)
- U4 pad 4: Net-(U1-S2) -> Net-(U1-S1)
- U4 pad 5: Net-(U1-S1) -> Net-(U1-S0)
- U4 pad 6: Net-(U1-S0) -> Net-(U2-COM)
- U4 pad 8: Net-(U2-S3) -> RX
- U4 pad 9: Net-(U2-S2) -> Net-(U2-~{E})

Commit message: マルツ行く前
Parts:
- added C1: C, Capacitor_SMD:C_0603_1608Metric, F.Cu at (-95.7, 252.8)
- added C2: C, Capacitor_SMD:C_0603_1608Metric, F.Cu at (-95.7, 255.3)
- added C3: C, Capacitor_SMD:C_0603_1608Metric, F.Cu at (-95.7, 257.8)
- added C4: C, Capacitor_SMD:C_0603_1608Metric, F.Cu at (-95.7, 260.3)
- added J1: Conn_01x09_Socket, Connector_PinSocket_2.54mm:PinSocket_1x09_P2.54mm_Horizontal, F.Cu at (-122.5, 246.1)
- added J2: Conn_01x09_Socket, Connector_PinSocket_2.54mm:PinSocket_1x09_P2.54mm_Horizontal, F.Cu at (-109.1, 246.1)
- added J3: Conn_01x09_Socket, Connector_PinHeader_2.54mm:PinHeader_1x09_P2.54mm_Horizontal, F.Cu at (-131.3, 221.1)
- added J4: Conn_01x09_Socket, Connector_PinHeader_2.54mm:PinHeader_1x09_P2.54mm_Horizontal, F.Cu at (-117.9, 221.1)
- added J5: Conn_01x09_Socket, Connector_PinHeader_2.54mm:PinHeader_1x09_P2.54mm_Horizontal, F.Cu at (-104.6, 221.1)
- added J6: Conn_01x09_Socket, Connector_PinHeader_2.54mm:PinHeader_1x09_P2.54mm_Horizontal, F.Cu at (-91.2, 221.1)
- added J7: Conn_01x02_Socket, Connector_JST:JST_XH_B2B-XH-AM_1x02_P2.50mm_Vertical, F.Cu at (-90.3, 254.9)
- added J8: Conn_01x04_Socket, Connector_JST:JST_XH_B4B-XH-AM_1x04_P2.50mm_Vertical, F.Cu at (-94.3, 247.1)
- added U1: 4051, Package_SO:TSSOP-16_4.4x5mm_P0.65mm, F.Cu at (-102.1, 247.1)
- added U2: 4051, Package_SO:TSSOP-16_4.4x5mm_P0.65mm, F.Cu at (-102.1, 253.6)
- added U3: 4051, Package_SO:TSSOP-16_4.4x5mm_P0.65mm, F.Cu at (-102.1, 260.2)
- added U4: 4051, Package_SO:TSSOP-16_4.4x5mm_P0.65mm, F.Cu at (-102.1, 266.8)
- J5: moved to B.Cu
- moved H1 57.6 mm to (65.0, 300.0)
- moved H2 36.5 mm to (-29.1, 316.5)
- moved J5 32.0 mm to (42.4, 257.6), turned to 45 degrees
- moved R1d1 8.91 mm to (67.4, 294.8), turned to 7.5 degrees
- moved Q6 8.89 mm to (8.88, 232.6), turned to -7.5 degrees
- moved Q5 8.89 mm to (26.0, 237.2), turned to -22.5 degrees
- moved Q4 8.89 mm to (41.4, 246.1), turned to -37.5 degrees
- moved Q3 8.88 mm to (53.9, 258.6), turned to -52.5 degrees
- moved Q2 8.88 mm to (62.8, 274.0), turned to -67.5 degrees
- moved Q1 8.88 mm to (67.4, 291.1), turned to -82.5 degrees
- moved R5 8.80 mm to (19.6, 235.6), turned to -112.5 degrees
- moved R3 8.79 mm to (49.0, 254.0), turned to -142.5 degrees
- moved R4 8.77 mm to (35.5, 243.0), turned to -127.5 degrees
- moved R6d1 8.59 mm to (12.3, 235.5), turned to 82.5 degrees
- moved R4d1 8.57 mm to (42.9, 250.4), turned to 52.5 degrees
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- renumbered U4 to U5
Connections:
- D10 pad 2: LED_5V_1 -> LED_5V_2
- D11 pad 2: LED_5V_1 -> LED_5V_2
- D12 pad 2: LED_5V_1 -> LED_5V_2
- D7 pad 2: LED_5V_1 -> LED_5V_2
- D8 pad 2: LED_5V_1 -> LED_5V_2
- D9 pad 2: LED_5V_1 -> LED_5V_2
- Q1 pad 1: Net-(J5-Pin_8) -> Net-(J1-Pin_9)
- Q10 pad 1: Net-(J6-Pin_5) -> Net-(J2-Pin_6)
- Q10 pad 2: GND1 -> GND2
- Q11 pad 1: Net-(J6-Pin_4) -> Net-(J2-Pin_5)
- Q11 pad 2: GND1 -> GND2
- Q12 pad 1: Net-(J6-Pin_3) -> Net-(J2-Pin_4)
- Q12 pad 2: GND1 -> GND2
- Q2 pad 1: Net-(J5-Pin_7) -> Net-(J1-Pin_8)
- Q3 pad 1: Net-(J5-Pin_6) -> Net-(J1-Pin_7)
- Q4 pad 1: Net-(J5-Pin_5) -> Net-(J1-Pin_6)
- Q5 pad 1: Net-(J5-Pin_4) -> Net-(J1-Pin_5)
- Q6 pad 1: Net-(J5-Pin_3) -> Net-(J1-Pin_4)
- Q7 pad 1: Net-(J6-Pin_8) -> Net-(J2-Pin_9)
- Q7 pad 2: GND1 -> GND2
- Q8 pad 1: Net-(J6-Pin_7) -> Net-(J2-Pin_8)
- Q8 pad 2: GND1 -> GND2
- Q9 pad 1: Net-(J6-Pin_6) -> Net-(J2-Pin_7)
- Q9 pad 2: GND1 -> GND2
- R1 pad 2: Net-(J5-Pin_8) -> Net-(J1-Pin_9)
- R10 pad 1: 3v3_1 -> 3v3_2
- R10 pad 2: Net-(J6-Pin_5) -> Net-(J2-Pin_6)
- R10d1 pad 2: GND1 -> GND2
- R11 pad 1: 3v3_1 -> 3v3_2
- R11 pad 2: Net-(J6-Pin_4) -> Net-(J2-Pin_5)
- R11d1 pad 2: GND1 -> GND2
- R12 pad 1: 3v3_1 -> 3v3_2
- R12 pad 2: Net-(J6-Pin_3) -> Net-(J2-Pin_4)
- R12d1 pad 2: GND1 -> GND2
- R2 pad 2: Net-(J5-Pin_7) -> Net-(J1-Pin_8)
- R3 pad 2: Net-(J5-Pin_6) -> Net-(J1-Pin_7)
- R4 pad 2: Net-(J5-Pin_5) -> Net-(J1-Pin_6)
- R5 pad 2: Net-(J5-Pin_4) -> Net-(J1-Pin_5)
- R6 pad 2: Net-(J5-Pin_3) -> Net-(J1-Pin_4)
- R7 pad 1: 3v3_1 -> 3v3_2
- R7 pad 2: Net-(J6-Pin_8) -> Net-(J2-Pin_9)
- R7d1 pad 2: GND1 -> GND2
- R8 pad 1: 3v3_1 -> 3v3_2
- R8 pad 2: Net-(J6-Pin_7) -> Net-(J2-Pin_8)
- R8d1 pad 2: GND1 -> GND2
- R9 pad 1: 3v3_1 -> 3v3_2
- R9 pad 2: Net-(J6-Pin_6) -> Net-(J2-Pin_7)
- R9d1 pad 2: GND1 -> GND2
- U5 pad 1: Net-(U1-COM) -> Net-(U1-X)
- U5 pad 10: Net-(U1-~{E}) -> Net-(U3-Inh)
- U5 pad 13: GND1 -> GND
- U5 pad 2: Net-(U1-S3) -> Net-(U1-A)
- U5 pad 3: Net-(U1-S2) -> Net-(U1-A)
- U5 pad 4: Net-(U1-S1) -> Net-(U1-A)
- U5 pad 5: Net-(U1-S0) -> Net-(U1-Inh)
- U5 pad 6: Net-(U2-COM) -> Net-(U2-Inh)
- U5 pad 9: Net-(U2-~{E}) -> Net-(U1-A)
Routing:
- net GND1: track 25.4 -> 7.04 mm, vias 2 -> 0
- net LED_5V_1: track 0.00 -> 14.6 mm, vias 0 -> 6
- net 3v3_1: track 6.72 -> 0.00 mm
- net Net-(J5-Pin_7): track 6.14 -> 0.00 mm
- net Net-(J5-Pin_8): track 5.76 -> 0.00 mm
- net Net-(D2-K): track 0.00 -> 3.81 mm
- net Net-(D1-K): track 0.00 -> 3.35 mm
- net Net-(D3-K): track 0.00 -> 3.16 mm
- net Net-(D5-K): track 0.00 -> 3.13 mm
- net Net-(D4-K): track 0.00 -> 3.05 mm
- net Net-(D6-K): track 0.00 -> 3.00 mm
- net Net-(J1-Pin_9): track 0.00 -> 2.58 mm
Other:
- outline, holes or cut-outs redrawn

Commit message: あきはばら
Parts:
- removed the J1 at (-215.6, 162.0)
- removed the J2 at (-187.4, 168.0)
- removed the J3 at (-112.0, 138.6)
- removed the J4 at (-137.7, 128.4)
- removed the J5 at (42.4, 257.6)
- removed the J6 at (-144.2, 349.0)
- removed the U1 at (-186.0, 151.4)
- removed the U2 at (-135.4, 150.0)
- J1: footprint Connector_PinSocket_2.54mm:PinSocket_1x09_P2.54mm_Horizontal -> Pinsocket_and_pinheader:PinSocket_1x09_P2.54mm_Horizontal_EDITED; moved to B.Cu
- J2: footprint Connector_PinSocket_2.54mm:PinSocket_1x09_P2.54mm_Horizontal -> Pinsocket_and_pinheader:PinSocket_1x09_P2.54mm_Horizontal_EDITED
- U5: footprint RF_Module:MCU_Seeed_ESP32C3 -> seeeduino:名称未設定
- moved J1 165.3 mm to (42.4, 257.6), turned to 45 degrees
- moved C1 146.3 mm to (-195.4, 145.8), turned to 180 degrees
- moved U1 138.3 mm to (-190.5, 140.7)
- moved C2 134.1 mm to (-195.7, 166.0), turned to 180 degrees
- moved U2 130.6 mm to (-193.4, 160.2)
- moved U3 129.1 mm to (-158.2, 143.9)
- moved C3 125.9 mm to (-160.5, 149.9), turned to 180 degrees
- moved J3 122.8 mm to (-222.6, 139.1), turned to 180 degrees
- moved J7 122.5 mm to (-183.2, 175.0), turned to 180 degrees
- moved U4 119.5 mm to (-157.4, 160.8)
- moved C4 113.4 mm to (-159.6, 166.6), turned to 180 degrees
- moved J4 110.5 mm to (-221.9, 183.8), turned to 180 degrees
- moved J5 104.8 mm to (-125.8, 118.5)
- moved J8 100.8 mm to (-165.1, 175.4), turned to 180 degrees
- moved J6 73.6 mm to (-123.0, 154.8)
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Connections:
- Q1 pad 1: Net-(J1-Pin_9) -> Net-(J1-Pin_4)
- Q2 pad 1: Net-(J1-Pin_8) -> Net-(J1-Pin_5)
- Q3 pad 1: Net-(J1-Pin_7) -> Net-(J1-Pin_6)
- Q4 pad 1: Net-(J1-Pin_6) -> Net-(J1-Pin_7)
- Q5 pad 1: Net-(J1-Pin_5) -> Net-(J1-Pin_8)
- Q6 pad 1: Net-(J1-Pin_4) -> Net-(J1-Pin_9)
- R1 pad 2: Net-(J1-Pin_9) -> Net-(J1-Pin_4)
- R2 pad 2: Net-(J1-Pin_8) -> Net-(J1-Pin_5)
- R3 pad 2: Net-(J1-Pin_7) -> Net-(J1-Pin_6)
- R4 pad 2: Net-(J1-Pin_6) -> Net-(J1-Pin_7)
- R5 pad 2: Net-(J1-Pin_5) -> Net-(J1-Pin_8)
- R6 pad 2: Net-(J1-Pin_4) -> Net-(J1-Pin_9)
Routing:
- net Net-(J1-Pin_4): track 0.00 -> 39.5 mm
- net Net-(J1-Pin_9): track 2.58 -> 36.0 mm
- net Net-(J1-Pin_5): track 0.00 -> 26.4 mm
- net 3v3_1: track 0.00 -> 24.8 mm, vias 0 -> 2
- net Net-(J1-Pin_8): track 0.00 -> 23.0 mm
- net Net-(J1-Pin_6): track 0.00 -> 13.9 mm
- net Net-(J1-Pin_7): track 0.00 -> 13.6 mm
- net GND1: track 7.04 -> 0.00 mm
- net LED_5V_1: track 14.6 -> 17.1 mm

Commit message: マイコン基板円形わお
Parts:
- added J10: Conn_01x03_Socket, Pinsocket_and_pinheader:PinHeader_1x03_P2.54mm_Vertical_EDITED, F.Cu at (2.00, 236.0)
- added J11: Conn_01x03_Socket, Pinsocket_and_pinheader:PinHeader_1x03_P2.54mm_Vertical_EDITED, F.Cu at (-101.0, 230.8)
- added J12: Conn_01x03_Socket, Pinsocket_and_pinheader:PinHeader_1x03_P2.54mm_Vertical_EDITED, F.Cu at (-117.0, 230.2)
- added J9: Conn_01x03_Socket, Pinsocket_and_pinheader:PinHeader_1x03_P2.54mm_Vertical_EDITED, F.Cu at (64.0, 298.0)
- added Q13: NMOS, Package_TO_SOT_THT:TO-251-3-1EP_Horizontal_TabDown, F.Cu at (-305.5, 144.6)
- added R13: R, Resistor_THT:R_Axial_DIN0207_L6.3mm_D2.5mm_P10.16mm_Horizontal, F.Cu at (-281.6, 142.5)
- added R14: R, Resistor_THT:R_Axial_DIN0207_L6.3mm_D2.5mm_P10.16mm_Horizontal, F.Cu at (-275.8, 147.1)
- J7: footprint Connector_JST:JST_XH_B2B-XH-AM_1x02_P2.50mm_Vertical -> Connector_JST:JST_XH_S2B-XH-A-1_1x02_P2.50mm_Horizontal
- J8: footprint Connector_JST:JST_XH_B4B-XH-AM_1x04_P2.50mm_Vertical -> Connector_JST:JST_XH_S4B-XH-A-1_1x04_P2.50mm_Horizontal
- moved J5 206.7 mm to (24.4, 260.6), turned to 45 degrees
- moved J3 145.3 mm to (-367.6, 147.7)
- moved U5 143.2 mm to (-299.5, 225.0)
- moved J6 141.9 mm to (-252.4, 213.0)
- moved J4 133.5 mm to (-343.6, 238.8)
- moved J7 120.1 mm to (-299.2, 143.9), turned to 0 degrees
- moved J8 91.7 mm to (-256.3, 184.2), turned to -90 degrees
- moved H2 85.9 mm to (21.8, 247.3)
- moved H1 25.1 mm to (52.7, 278.2)
- moved R6 0.98 mm to (5.46, 232.1), turned to -97.5 degrees
Connections:
- U5 pad 11: unconnected-(U5-10-Pad11) -> Net-(U5-10)
Routing:
- net LED_5V_1: track 17.1 -> 32.1 mm
- net 3v3_1: track 24.8 -> 34.7 mm
Other:
- board size 336.4 x 337.8 mm -> 616 x 338.6 mm
- board text added: "URAWA BEOLSAE 2025"

Commit message: kicad欄センサーエラー0まで
Parts:
- added H5: MountingHole, MountingHole:MountingHole_3.2mm_M3, F.Cu at (155.7, 97.8)
- added H6: MountingHole, MountingHole:MountingHole_3.2mm_M3, F.Cu at (244.3, 97.8)
- added H7: MountingHole, MountingHole:MountingHole_3.2mm_M3, F.Cu at (200.0, 135.0)
- added H8: MountingHole, MountingHole:MountingHole_3.2mm_M3, F.Cu at (218.0, 58.8)
- added H9: MountingHole, MountingHole:MountingHole_3.2mm_M3, F.Cu at (182.0, 58.8)
- C1, C2, C3, C4, J2, J7, J8, Q13, R13, R14, U5: moved to B.Cu
- J3, J4, J5, J6: footprint Connector_PinHeader_2.54mm:PinHeader_1x09_P2.54mm_Horizontal -> Pinsocket_and_pinheader:PinHeader_1x09_P2.54mm_Horizontal_EDITED; moved to B.Cu
- U1, U2, U3, U4: footprint Package_SO:TSSOP-16_4.4x5mm_P0.65mm -> Pinsocket_and_pinheader:CERDIP-16_W7.62mm_SideBrazed_LongPads_pin_EDITED; moved to B.Cu
- moved J3 606.7 mm to (232.4, 57.6), turned to 45 degrees
- moved J4 587.6 mm to (232.4, 122.4), turned to -45 degrees
- moved Q13 522.3 mm to (207.7, 47.4), turned to 75 degrees
- moved J7 509.9 mm to (201.4, 46.7), turned to 180 degrees
- moved U5 505.2 mm to (190.0, 100.0), turned to 180 degrees
- moved R13 475.7 mm to (184.0, 45.2), turned to 10 degrees
- moved J8 469.8 mm to (205.0, 95.0), turned to 0 degrees
- moved R14 469.2 mm to (183.1, 49.3), turned to 10 degrees
- moved J6 429.7 mm to (167.6, 122.4), turned to -135 degrees
- moved C1 425.9 mm to (227.0, 91.4)
- moved U1 422.2 mm to (230.0, 103.0)
- moved C2 408.5 mm to (209.1, 111.2)
- moved U2 407.1 mm to (212.0, 123.0)
- moved D10 384.4 mm to (93.8, 63.1), turned to 142.5 degrees
- moved D11 382.7 mm to (79.1, 54.6), turned to 157.5 degrees
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Connections:
- Q10 pad 1: Net-(J2-Pin_6) -> Net-(J2-Pin_7)
- Q11 pad 1: Net-(J2-Pin_5) -> Net-(J2-Pin_8)
- Q12 pad 1: Net-(J2-Pin_4) -> Net-(J2-Pin_9)
- Q7 pad 1: Net-(J2-Pin_9) -> Net-(J2-Pin_4)
- Q8 pad 1: Net-(J2-Pin_8) -> Net-(J2-Pin_5)
- Q9 pad 1: Net-(J2-Pin_7) -> Net-(J2-Pin_6)
- R10 pad 2: Net-(J2-Pin_6) -> Net-(J2-Pin_7)
- R11 pad 2: Net-(J2-Pin_5) -> Net-(J2-Pin_8)
- R12 pad 2: Net-(J2-Pin_4) -> Net-(J2-Pin_9)
- R7 pad 2: Net-(J2-Pin_9) -> Net-(J2-Pin_4)
- R8 pad 2: Net-(J2-Pin_8) -> Net-(J2-Pin_5)
- R9 pad 2: Net-(J2-Pin_7) -> Net-(J2-Pin_6)
- U1 pad 1: Net-(J3-Pin_5) -> unconnected-(U1-X4-Pad1)
- U1 pad 10: Net-(U1-A) -> Net-(U1-B)
- U1 pad 12: Net-(J3-Pin_6) -> Net-(J3-Pin_7)
- U1 pad 13: Net-(J3-Pin_9) -> Net-(J3-Pin_6)
- U1 pad 14: Net-(J3-Pin_8) -> Net-(J3-Pin_5)
- U1 pad 15: Net-(J3-Pin_7) -> Net-(J3-Pin_4)
- U1 pad 4: unconnected-(U1-X7-Pad4) -> Net-(J3-Pin_8)
- U1 pad 5: Net-(J3-Pin_4) -> Net-(J3-Pin_9)
- U1 pad 9: Net-(U1-A) -> Net-(U1-C)
- U2 pad 1: Net-(J4-Pin_5) -> unconnected-(U2-X4-Pad1)
- U2 pad 10: Net-(U1-A) -> Net-(U1-B)
- U2 pad 12: Net-(J4-Pin_6) -> Net-(J4-Pin_7)
- U2 pad 13: Net-(J4-Pin_9) -> Net-(J4-Pin_6)
- U2 pad 14: Net-(J4-Pin_8) -> Net-(J4-Pin_5)
- U2 pad 15: Net-(J4-Pin_7) -> Net-(J4-Pin_4)
- U2 pad 4: unconnected-(U2-X7-Pad4) -> Net-(J4-Pin_8)
- U2 pad 5: Net-(J4-Pin_4) -> Net-(J4-Pin_9)
- U2 pad 9: Net-(U1-A) -> Net-(U1-C)
- U3 pad 1: Net-(J5-Pin_5) -> Net-(J5-Pin_4)
- U3 pad 10: Net-(U1-A) -> Net-(U1-B)
- U3 pad 12: Net-(J5-Pin_6) -> Net-(J5-Pin_9)
- U3 pad 13: Net-(J5-Pin_9) -> Net-(J5-Pin_8)
- U3 pad 14: Net-(J5-Pin_8) -> Net-(J5-Pin_7)
- U3 pad 15: Net-(J5-Pin_7) -> Net-(J5-Pin_6)
- U3 pad 2: unconnected-(U3-X6-Pad2) -> Net-(J5-Pin_5)
- U3 pad 5: Net-(J5-Pin_4) -> unconnected-(U3-X5-Pad5)
- U3 pad 9: Net-(U1-A) -> Net-(U1-C)
- U4 pad 1: Net-(J6-Pin_5) -> Net-(J6-Pin_4)
- U4 pad 10: Net-(U1-A) -> Net-(U1-B)
- U4 pad 12: Net-(J6-Pin_6) -> Net-(J6-Pin_9)
- U4 pad 13: Net-(J6-Pin_9) -> Net-(J6-Pin_8)
- U4 pad 14: Net-(J6-Pin_8) -> Net-(J6-Pin_7)
- U4 pad 15: Net-(J6-Pin_7) -> Net-(J6-Pin_6)
- U4 pad 2: unconnected-(U4-X6-Pad2) -> Net-(J6-Pin_5)
- U4 pad 5: Net-(J6-Pin_4) -> unconnected-(U4-X5-Pad5)
- U4 pad 6: Net-(U1-A) -> Net-(U4-Inh)
- U4 pad 9: Net-(U1-A) -> Net-(U1-C)
- U5 pad 14: unconnected-(U5-VCC-Pad14) -> VCC
- U5 pad 3: Net-(U1-A) -> Net-(U1-B)
- U5 pad 4: Net-(U1-A) -> Net-(U1-C)
- U5 pad 9: Net-(U1-A) -> Net-(U4-Inh)
Routing:
- net GND: track 0.00 -> 439.7 mm, vias 0 -> 12
- net seed_3v3: track 0.00 -> 307.7 mm, vias 0 -> 4
- net GND1: track 0.00 -> 161.9 mm, vias 0 -> 17
- net GND2: track 0.00 -> 156.6 mm, vias 0 -> 16
- net Net-(U1-X): track 0.00 -> 154.6 mm, vias 0 -> 4
- net Net-(U1-A): track 0.00 -> 136.3 mm, vias 0 -> 4
- net Net-(U1-B): track 0.00 -> 131.4 mm, vias 0 -> 2
- net Net-(U1-C): track 0.00 -> 125.9 mm, vias 0 -> 3
- net LED_5V: track 0.00 -> 122.0 mm, vias 0 -> 2
- net Net-(U5-10): track 0.00 -> 47.0 mm, vias 0 -> 1
- net RX: track 0.00 -> 43.1 mm
- net Net-(J4-Pin_9): track 0.00 -> 34.1 mm
- net LED_5V_2: track 0.00 -> 33.7 mm, vias 0 -> 6
- net Net-(U4-Inh): track 0.00 -> 33.1 mm, vias 0 -> 1
- net Net-(J4-Pin_8): track 0.00 -> 32.6 mm
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- added copper zone on B.Cu, net GND
- added copper zone on F.Cu, net GND
- added copper zone on B.Cu, net GND1
- added copper zone on F.Cu, net GND1
- added copper zone on B.Cu, net GND2
- added copper zone on F.Cu, net GND2
Other:
- board size 616 x 338.6 mm -> 217.1 x 100 mm
- board text added: "2025-2026"
- board text added: "URAWA BEOLSAE"
- board text added: "unit1"
- board text added: "unit2"
- board text removed: "URAWA BEOLSAE 2025"
- board text removed: "外側r=70, 内側r=55の場合"
- board text removed: "外側r=70, 内側r=60の場合 +角削る"
