File: kiCad/LineSensor_Block_prot2/LineSensor_Block_prot2.kicad_sch (KiCad schematic)
At the start: 69 parts, among them J1 Conn_01x09_Socket, J2 Conn_01x09_Socket, J3 Conn_01x09_Socket, J4 Conn_01x09_Socket, J5 Conn_01x09_Socket, J6 Conn_01x09_Socket, J7 Conn_01x02_Socket, J8 Conn_01x04_Socket, Q1 Q_Photo_NPN, Q10 Q_Photo_NPN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

Commit message: マルツ行く前
Parts:
- C1, C2, C3, C4: footprint (none) -> Capacitor_SMD:C_0603_1608Metric
- J1, J2: footprint (none) -> Connector_PinSocket_2.54mm:PinSocket_1x09_P2.54mm_Horizontal
- J3, J4, J5, J6: footprint (none) -> Connector_PinHeader_2.54mm:PinHeader_1x09_P2.54mm_Horizontal
- J7: footprint (none) -> Connector_JST:JST_XH_B2B-XH-AM_1x02_P2.50mm_Vertical
- J8: footprint (none) -> Connector_JST:JST_XH_B4B-XH-AM_1x04_P2.50mm_Vertical
- U1, U2, U3, U4: footprint (none) -> Package_SO:TSSOP-16_4.4x5mm_P0.65mm
Changed lines of the file:
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@@
 			)
 		)
-		(property "Footprint" ""
+		(property "Footprint" "Connector_PinSocket_2.54mm:PinSocket_1x09_P2.54mm_Horizontal"
 			(at 406.4 267.97 0)
 			(effects
@@
 			)
 		)
-		(property "Footprint" ""
+		(property "Footprint" "Package_SO:TSSOP-16_4.4x5mm_P0.65mm"
 			(at 205.74 101.6 0)
 			(effects
@@
 			)
 		)
-		(property "Footprint" ""
+		(property "Footprint" "Connector_JST:JST_XH_B2B-XH-AM_1x02_P2.50mm_Vertical"
 			(at 316.23 101.6 0)
 			(effects
@@
 			)
 		)
-		(property "Footprint" ""
+		(property "Footprint" "Capacitor_SMD:C_0603_1608Metric"
 			(at 213.36 71.4248 0)
 			(effects
@@
 			)
 		)
-		(property "Footprint" ""
+		(property "Footprint" "Package_SO:TSSOP-16_4.4x5mm_P0.65mm"
 			(at 205.74 184.15 0)
 			(effects
@@
 			)
 		)
-		(property "Footprint" ""
+		(property "Footprint" "Connector_PinHeader_2.54mm:PinHeader_1x09_P2.54mm_Horizontal"
 			(at 154.94 179.07 0)
 			(effects
@@
 			)
 		)
-		(property "Footprint" ""
+		(property "Footprint" "Capacitor_SMD:C_0603_1608Metric"
 			(at 267.97 153.3652 0)
 			(effects
@@
 			)
 		)
-		(property "Footprint" ""
+		(property "Footprint" "Connector_JST:JST_XH_B4B-XH-AM_1x04_P2.50mm_Vertical"
 			(at 314.96 118.11 0)
 			(effects
@@
 			)
 		)
-		(property "Footprint" ""
+		(property "Footprint" "Connector_PinSocket_2.54mm:PinSocket_1x09_P2.54mm_Horizontal"
 			(at 420.37 86.36 0)
 			(effects
@@
 			)
 		)
-		(property "Footprint" ""
+		(property "Footprint" "Package_SO:TSSOP-16_4.4x5mm_P0.65mm"
 			(at 276.86 185.42 0)
 			(effects
@@
 			)
 		)
-		(property "Footprint" ""
+		(property "Footprint" "Capacitor_SMD:C_0603_1608Metric"
 			(at 283.21 63.8048 0)
 			(effects
@@
 			)
 		)
-		(property "Footprint" ""
+		(property "Footprint" "Package_SO:TSSOP-16_4.4x5mm_P0.65mm"
 			(at 275.59 92.71 0)
 			(effects
@@
 			)
 		)
-		(property "Footprint" ""
+		(property "Footprint" "Connector_PinHeader_2.54mm:PinHeader_1x09_P2.54mm_Horizontal"
 			(at 229.87 180.34 0)
 			(effects
@@
 			)
 		)
-		(property "Footprint" ""
+		(property "Footprint" "Connector_PinHeader_2.54mm:PinHeader_1x09_P2.54mm_Horizontal"
 			(at 152.4 96.52 0)
 			(effects
@@
 			)
 		)
-		(property "Footprint" ""
+		(property "Footprint" "Connector_PinHeader_2.54mm:PinHeader_1x09_P2.54mm_Horizontal"
 			(at 233.68 87.63 0)
 			(effects
@@
 			)
 		)
-		(property "Footprint" ""
+		(property "Footprint" "Capacitor_SMD:C_0603_1608Metric"
 			(at 198.12 154.6352 0)
 			(effects

Commit message: あきはばら
Parts:
- J1, J2: footprint Connector_PinSocket_2.54mm:PinSocket_1x09_P2.54mm_Horizontal -> Pinsocket_and_pinheader:PinSocket_1x09_P2.54mm_Horizontal_EDITED
- U5: footprint RF_Module:MCU_Seeed_ESP32C3 -> seeeduino:名称未設定
Connections:
- net at Q4.1 (C), R4.2: now also J1.7 (Pin_7); no longer J1.6 (Pin_6)
- net at Q6.1 (C), R6.2: now also J1.9 (Pin_9); no longer J1.4 (Pin_4)
- net at Q5.1 (C), R5.2: now also J1.8 (Pin_8); no longer J1.5 (Pin_5)
- net at Q3.1 (C), R3.2: now also J1.6 (Pin_6); no longer J1.7 (Pin_7)
- net at Q2.1 (C), R2.2: now also J1.5 (Pin_5); no longer J1.8 (Pin_8)
- net at Q1.1 (C), R1.2: now also J1.4 (Pin_4); no longer J1.9 (Pin_9)
Changed lines of the file:
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@@
 	)
 	(junction
+		(at 420.37 49.53)
+		(diameter 0)
+		(color 0 0 0 0)
+	)
+	(junction
 		(at 474.98 224.79)
 		(diameter 0)
@@
 	)
 	(junction
+		(at 417.83 52.07)
+		(diameter 0)
+		(color 0 0 0 0)
+	)
+	(junction
 		(at 463.55 69.85)
 		(diameter 0)
@@
 	(wire
 		(pts
+			(xy 415.29 52.07) (xy 417.83 52.07)
+		)
+		(stroke
+			(width 0)
+			(type default)
+		)
+	)
+	(wire
+		(pts
 			(xy 193.04 191.77) (xy 193.04 194.31)
 		)
@@
 	(wire
 		(pts
-			(xy 417.83 81.28) (xy 417.83 54.61)
-		)
-		(stroke
-			(width 0)
-			(type default)
-		)
-	)
-	(wire
-		(pts
 			(xy 264.16 200.66) (xy 254 200.66)
 		)
@@
 	(wire
 		(pts
+			(xy 410.21 59.69) (xy 525.78 59.69)
+		)
+		(stroke
+			(width 0)
+			(type default)
+		)
+	)
+	(wire
+		(pts
 			(xy 179.07 194.31) (xy 193.04 194.31)
 		)
@@
 	(wire
 		(pts
-			(xy 412.75 49.53) (xy 429.26 49.53)
+			(xy 412.75 49.53) (xy 420.37 49.53)
 		)
 		(stroke
@@
 	(wire
 		(pts
-			(xy 420.37 57.15) (xy 499.11 57.15)
+			(xy 234.95 180.34) (xy 264.16 180.34)
 		)
 		(stroke
@@
 	(wire
 		(pts
-			(xy 234.95 180.34) (xy 264.16 180.34)
+			(xy 485.14 214.63) (xy 474.98 214.63)
 		)
 		(stroke
@@
 	(wire
 		(pts
-			(xy 485.14 214.63) (xy 474.98 214.63)
+			(xy 396.24 262.89) (xy 396.24 214.63)
 		)
 		(stroke
@@
 	(wire
 		(pts
-			(xy 396.24 262.89) (xy 396.24 214.63)
+			(xy 422.91 81.28) (xy 422.91 48.26)
 		)
 		(stroke
@@
 	(wire
 		(pts
-			(xy 422.91 59.69) (xy 525.78 59.69)
+			(xy 420.37 49.53) (xy 429.26 49.53)
 		)
 		(stroke
@@
 	(wire
 		(pts
-			(xy 453.39 30.48) (xy 443.23 30.48)
+			(xy 417.83 52.07) (xy 417.83 81.28)
 		)
 		(stroke
@@
 	(wire
 		(pts
-			(xy 452.12 224.79) (xy 474.98 224.79)
+			(xy 453.39 30.48) (xy 443.23 30.48)
 		)
 		(stroke
@@
 	(wire
 		(pts
-			(xy 330.2 222.25) (xy 330.2 147.32)
+			(xy 452.12 224.79) (xy 474.98 224.79)
 		)
 		(stroke
@@
 	(wire
 		(pts
-			(xy 398.78 228.6) (xy 417.83 228.6)
+			(xy 330.2 222.25) (xy 330.2 147.32)
 		)
 		(stroke
@@
 	(wire
 		(pts
-			(xy 160.02 173.99) (xy 193.04 173.99)
+			(xy 398.78 228.6) (xy 417.83 228.6)
 		)
 		(stroke
@@
 	(wire
 		(pts
-			(xy 410.21 81.28) (xy 410.21 30.48)
+			(xy 160.02 173.99) (xy 193.04 173.99)
 		)
 		(stroke
@@
 	(wire
 		(pts
+			(xy 420.37 49.53) (xy 420.37 81.28)
+		)
+		(stroke
+			(width 0)
+			(type default)
+		)
+	)
+	(wire
+		(pts
+			(xy 412.75 57.15) (xy 499.11 57.15)
+		)
+		(stroke
+			(width 0)
+			(type default)
+		)
+	)
+	(wire
+		(pts
 			(xy 406.4 262.89) (xy 406.4 236.22)
 		)
@@
 	(wire
 		(pts
-			(xy 417.83 54.61) (xy 476.25 54.61)
+			(xy 179.07 111.76) (xy 179.07 137.16)
 		)
 		(stroke
@@
 	(wire
 		(pts
-			(xy 179.07 111.76) (xy 179.07 137.16)
+			(xy 525.78 30.48) (xy 511.81 30.48)
 		)
 		(stroke
@@
 	(wire
 		(pts
-			(xy 525.78 30.48) (xy 511.81 30.48)
+			(xy 238.76 92.71) (xy 260.35 92.71)
 		)
 		(stroke
@@
 	(wire
 		(pts
-			(xy 238.76 92.71) (xy 260.35 92.71)
+			(xy 184.15 142.24) (xy 254 142.24)
 		)
 		(stroke
@@
 	(wire
 		(pts
-			(xy 415.29 52.07) (xy 453.39 52.07)
+			(xy 462.28 233.68) (xy 462.28 214.63)
 		)
 		(stroke
@@
 	(wire
 		(pts
-			(xy 184.15 142.24) (xy 254 142.24)
+			(xy 320.04 137.16) (xy 337.82 137.16)
 		)
 		(stroke
@@
 	(wire
 		(pts
-			(xy 462.28 233.68) (xy 462.28 214.63)
+			(xy 410.21 48.26) (xy 410.21 30.48)
 		)
 		(stroke
@@
 	(wire
 		(pts
-			(xy 320.04 137.16) (xy 337.82 137.16)
+			(xy 488.95 29.21) (xy 488.95 30.48)
 		)
 		(stroke
@@
 	(wire
 		(pts
-			(xy 488.95 29.21) (xy 488.95 30.48)
+			(xy 417.83 52.07) (xy 453.39 52.07)
 		)
 		(stroke
@@
 	(wire
 		(pts
-			(xy 179.07 137.16) (xy 179.07 194.31)
+			(xy 415.29 54.61) (xy 476.25 54.61)
 		)
 		(stroke
@@
 	(wire
 		(pts
-			(xy 234.95 185.42) (xy 259.08 185.42)
+			(xy 179.07 137.16) (xy 179.07 194.31)
 		)
 		(stroke
@@
 	(wire
 		(pts
-			(xy 415.29 81.28) (xy 415.29 52.07)
+			(xy 234.95 185.42) (xy 259.08 185.42)
 		)
 		(stroke
@@
 	(wire
 		(pts
+			(xy 412.75 81.28) (xy 412.75 57.15)
+		)
+		(stroke
+			(width 0)
+			(type default)
+		)
+	)
+	(wire
+		(pts
 			(xy 275.59 64.77) (xy 275.59 69.85)
 		)
@@
 	(wire
 		(pts
-			(xy 422.91 81.28) (xy 422.91 59.69)
-		)
-		(stroke
-			(width 0)
-			(type default)
-		)
-	)
-	(wire
-		(pts
 			(xy 508 85.09) (xy 518.16 85.09)
 		)
@@
 	(wire
 		(pts
-			(xy 420.37 81.28) (xy 420.37 57.15)
+			(xy 443.23 29.21) (xy 443.23 30.48)
 		)
 		(stroke
@@
 	(wire
 		(pts
-			(xy 443.23 29.21) (xy 443.23 30.48)
+			(xy 422.91 48.26) (xy 410.21 48.26)
 		)
 		(stroke
@@
 	(wire
 		(pts
+			(xy 410.21 59.69) (xy 410.21 81.28)
+		)
+		(stroke
+			(width 0)
+			(type default)
+		)
+	)
+	(wire
+		(pts
 			(xy 462.28 214.63) (xy 452.12 214.63)
 		)
@@
 	(wire
 		(pts
-			(xy 412.75 81.28) (xy 412.75 49.53)
+			(xy 415.29 54.61) (xy 415.29 81.28)
 		)
 		(stroke
@@
 			)
 		)
-		(property "Footprint" "Connector_PinSocket_2.54mm:PinSocket_1x09_P2.54mm_Horizontal"
+		(property "Footprint" "Pinsocket_and_pinheader:PinSocket_1x09_P2.54mm_Horizontal_EDITED"
 			(at 406.4 267.97 0)
 			(effects
@@
 			)
 		)
-		(property "Footprint" "RF_Module:MCU_Seeed_ESP32C3"
+		(property "Footprint" "seeeduino:名称未設定"
 			(at 309.88 139.7 0)
 			(effects
@@
 			)
 		)
-		(property "Footprint" "Connector_PinSocket_2.54mm:PinSocket_1x09_P2.54mm_Horizontal"
+		(property "Footprint" "Pinsocket_and_pinheader:PinSocket_1x09_P2.54mm_Horizontal_EDITED"
 			(at 420.37 86.36 0)
 			(effects

Commit message: マイコン基板円形わお
Parts:
- added J10, J11, J12, J9: Conn_01x03_Socket, Pinsocket_and_pinheader:PinHeader_1x03_P2.54mm_Vertical_EDITED, symbol Connector:Conn_01x03_Socket
- added Q13: NMOS, Package_TO_SOT_THT:TO-251-3-1EP_Horizontal_TabDown, symbol Simulation_SPICE:NMOS
- added R13, R14: R, Resistor_THT:R_Axial_DIN0207_L6.3mm_D2.5mm_P10.16mm_Horizontal, symbol Device:R
- J7: footprint Connector_JST:JST_XH_B2B-XH-AM_1x02_P2.50mm_Vertical -> Connector_JST:JST_XH_S2B-XH-A-1_1x02_P2.50mm_Horizontal
- J8: footprint Connector_JST:JST_XH_B4B-XH-AM_1x04_P2.50mm_Vertical -> Connector_JST:JST_XH_S4B-XH-A-1_1x04_P2.50mm_Horizontal
Connections:
- net 3v3_1: now also J10.2 (Pin_2), J9.2 (Pin_2)
- net 3v3_2: now also J11.2 (Pin_2), J12.2 (Pin_2)
- net GND: now also Q13.3 (S), R14.2
- net GND1: now also J10.1 (Pin_1), J9.1 (Pin_1)
- net GND2: now also J11.1 (Pin_1), J12.1 (Pin_1)
- net LED_5V: now also Q13.1 (D)
- net LED_5V_1: now also J10.3 (Pin_3), J9.3 (Pin_3)
- net LED_5V_2: now also J11.3 (Pin_3), J12.3 (Pin_3)
- net at U5.11 (10): now also R13.2
- new net: Q13.2 (G), R13.1, R14.1

Commit message: kicad欄センサーエラー0まで
Parts:
- added H5, H6, H7, H8, H9: MountingHole, MountingHole:MountingHole_3.2mm_M3, symbol Mechanical:MountingHole
- J3, J4, J5, J6: footprint Connector_PinHeader_2.54mm:PinHeader_1x09_P2.54mm_Horizontal -> Pinsocket_and_pinheader:PinHeader_1x09_P2.54mm_Horizontal_EDITED
- U1, U2, U3, U4: footprint Package_SO:TSSOP-16_4.4x5mm_P0.65mm -> Pinsocket_and_pinheader:CERDIP-16_W7.62mm_SideBrazed_LongPads_pin_EDITED
Connections:
- net VCC: now also U5.14 (VCC)
- net at Q12.1 (C), R12.2: now also J2.9 (Pin_9); no longer J2.4 (Pin_4)
- net at Q11.1 (C), R11.2: now also J2.8 (Pin_8); no longer J2.5 (Pin_5)
- net at Q10.1 (C), R10.2: now also J2.7 (Pin_7); no longer J2.6 (Pin_6)
- net at Q9.1 (C), R9.2: now also J2.6 (Pin_6); no longer J2.7 (Pin_7)
- net at Q8.1 (C), R8.2: now also J2.5 (Pin_5); no longer J2.8 (Pin_8)
- net at Q7.1 (C), R7.2: now also J2.4 (Pin_4); no longer J2.9 (Pin_9)
- net at U3.1 (X4): now also J5.4 (Pin_4); no longer J5.5 (Pin_5)
- net at U3.12 (X3): now also J5.9 (Pin_9); no longer J5.6 (Pin_6)
- net at U3.13 (X0): now also J5.8 (Pin_8); no longer J5.9 (Pin_9)
- net at U3.14 (X1): now also J5.7 (Pin_7); no longer J5.8 (Pin_8)
- net at U3.15 (X2): now also J5.6 (Pin_6); no longer J5.7 (Pin_7)
- net at U3.2 (X6): now also J5.5 (Pin_5)
- net at U3.5 (X5): no longer J5.4 (Pin_4)
- net at U4.1 (X4): now also J6.4 (Pin_4); no longer J6.5 (Pin_5)
- net at U4.12 (X3): now also J6.9 (Pin_9); no longer J6.6 (Pin_6)
- net at U4.13 (X0): now also J6.8 (Pin_8); no longer J6.9 (Pin_9)
- net at U4.14 (X1): now also J6.7 (Pin_7); no longer J6.8 (Pin_8)
- net at U4.15 (X2): now also J6.6 (Pin_6); no longer J6.7 (Pin_7)
- net at U4.2 (X6): now also J6.5 (Pin_5)
- net at U4.5 (X5): no longer J6.4 (Pin_4)
- net at U2.1 (X4): no longer J4.5 (Pin_5)
- net at U2.12 (X3): now also J4.7 (Pin_7); no longer J4.6 (Pin_6)
- net at U2.13 (X0): now also J4.6 (Pin_6); no longer J4.9 (Pin_9)
- net at U2.14 (X1): now also J4.5 (Pin_5); no longer J4.8 (Pin_8)
- net at U2.15 (X2): now also J4.4 (Pin_4); no longer J4.7 (Pin_7)
- net at U2.4 (X7): now also J4.8 (Pin_8)
- net at U2.5 (X5): now also J4.9 (Pin_9); no longer J4.4 (Pin_4)
- net at U1.1 (X4): no longer J3.5 (Pin_5)
- net at U1.12 (X3): now also J3.7 (Pin_7); no longer J3.6 (Pin_6)
- net at U1.13 (X0): now also J3.6 (Pin_6); no longer J3.9 (Pin_9)
- net at U1.14 (X1): now also J3.5 (Pin_5); no longer J3.8 (Pin_8)
- net at U1.15 (X2): now also J3.4 (Pin_4); no longer J3.7 (Pin_7)
- net at U1.4 (X7): now also J3.8 (Pin_8)
- net at U1.5 (X5): now also J3.9 (Pin_9); no longer J3.4 (Pin_4)
- new net: U1.10 (B), U2.10 (B), U3.10 (B), U4.10 (B), U5.3 (2)
- new net: U1.11 (A), U2.11 (A), U3.11 (A), U4.11 (A), U5.2 (1)
- new net: U1.9 (C), U2.9 (C), U3.9 (C), U4.9 (C), U5.4 (3)
- new net: U4.6 (Inh), U5.9 (8)
Other:
- moved on the sheet: H1, H2, H3, H4, J4, J6
