File: KiCad/Linesensor_Japan_prot1/Linesensor_Japan_prot1.kicad_pcb (KiCad board)
At the start: 2 copper layers, 140 x 140 mm, 140 parts, among them J1 Conn_01x04_Socket, J2 Conn_01x02_Socket, Q1 Q_Photo_NPN, Q10 Q_Photo_NPN, Q11 Q_Photo_NPN, Q12 Q_Photo_NPN, Q13 Q_Photo_NPN, Q14 Q_Photo_NPN, Q15 Q_Photo_NPN, Q16 Q_Photo_NPN, Q17 Q_Photo_NPN, Q18 Q_Photo_NPN, Q19 Q_Photo_NPN, Q2 Q_Photo_NPN, Q20 Q_Photo_NPN, Q21 Q_Photo_NPN, Q22 Q_Photo_NPN, Q23 Q_Photo_NPN, Q24 Q_Photo_NPN, Q25 Q_Photo_NPN, Q26 Q_Photo_NPN, Q27 Q_Photo_NPN, Q28 Q_Photo_NPN, Q29 Q_Photo_NPN, Q3 Q_Photo_NPN, Q30 Q_Photo_NPN, Q31 Q_Photo_NPN, Q32 Q_Photo_NPN, Q33 Q_NMOS, Q4 Q_Photo_NPN, Q5 Q_Photo_NPN, Q6 Q_Photo_NPN, Q7 Q_Photo_NPN, Q8 Q_Photo_NPN, Q9 Q_Photo_NPN, U1 CD74HC4067SM, U2 CD74HC4067SM

Commit message: ラインセンサーprot1ほぼ完成
Parts:
- added G***: LOGO, JLCPCB:JLCPCB, F.Cu at (262.7, 64.2)
- added G***: LOGO, JLCPCB:JCLPCB_15.1x4.4, F.Cu at (123.0, 149.4)
- added G***: LOGO, JLCPCB:JLCPCB, F.Cu at (264.2, 23.1)
- moved Q33 47.9 mm to (80.5, 145.6), turned to 0 degrees
- moved R74 47.3 mm to (66.0, 141.8), turned to -30 degrees
- moved J1 38.2 mm to (115.6, 139.9)
- moved R73 33.2 mm to (77.2, 153.7), turned to 150 degrees
- moved J2 32.5 mm to (80.5, 140.8)
- moved U3 14.7 mm to (100.2, 151.1)
- moved C1 13.8 mm to (45.1, 107.4), turned to 0 degrees
- moved C3 9.36 mm to (107.9, 140.0)
- moved C4 5.80 mm to (89.6, 152.4)
- moved C2 3.69 mm to (156.2, 93.0)
- moved U2 0.88 mm to (42.8, 100.0), turned to -90 degrees
- turned U1 to 90 degrees
Connections:
- Q2 pad 2: unconnected-(Q2-E-Pad2) -> GND
- U1 pad 16: unconnected-(U1-I15-Pad16) -> Net-(Q6-C)
- U1 pad 17: unconnected-(U1-I14-Pad17) -> Net-(Q5-C)
- U1 pad 18: unconnected-(U1-I13-Pad18) -> Net-(Q4-C)
- U1 pad 19: unconnected-(U1-I12-Pad19) -> Net-(Q3-C)
- U1 pad 2: unconnected-(U1-I7-Pad2) -> Net-(Q26-C)
- U1 pad 20: unconnected-(U1-I11-Pad20) -> Net-(Q2-C)
- U1 pad 21: unconnected-(U1-I10-Pad21) -> Net-(Q7-C)
- U1 pad 22: unconnected-(U1-I9-Pad22) -> Net-(Q8-C)
- U1 pad 23: unconnected-(U1-I8-Pad23) -> Net-(Q9-C)
- U1 pad 3: Net-(Q2-C) -> Net-(Q1-C)
- U1 pad 4: Net-(Q1-C) -> Net-(Q32-C)
- U1 pad 5: unconnected-(U1-I4-Pad5) -> Net-(Q31-C)
- U1 pad 6: unconnected-(U1-I3-Pad6) -> Net-(Q30-C)
- U1 pad 7: unconnected-(U1-I2-Pad7) -> Net-(Q29-C)
- U1 pad 8: unconnected-(U1-I1-Pad8) -> Net-(Q28-C)
- U1 pad 9: unconnected-(U1-I0-Pad9) -> Net-(Q27-C)
- U2 pad 16: unconnected-(U2-I15-Pad16) -> Net-(Q25-C)
- U2 pad 17: unconnected-(U2-I14-Pad17) -> Net-(Q24-C)
- U2 pad 18: unconnected-(U2-I13-Pad18) -> Net-(Q23-C)
- U2 pad 19: unconnected-(U2-I12-Pad19) -> Net-(Q22-C)
- U2 pad 2: unconnected-(U2-I7-Pad2) -> Net-(Q17-C)
- U2 pad 20: unconnected-(U2-I11-Pad20) -> Net-(Q21-C)
- U2 pad 21: unconnected-(U2-I10-Pad21) -> Net-(Q20-C)
- U2 pad 22: unconnected-(U2-I9-Pad22) -> Net-(Q19-C)
- U2 pad 23: unconnected-(U2-I8-Pad23) -> Net-(Q18-C)
- U2 pad 3: unconnected-(U2-I6-Pad3) -> Net-(Q16-C)
- U2 pad 4: unconnected-(U2-I5-Pad4) -> Net-(Q15-C)
- U2 pad 5: unconnected-(U2-I4-Pad5) -> Net-(Q14-C)
- U2 pad 6: unconnected-(U2-I3-Pad6) -> Net-(Q10-C)
- U2 pad 7: unconnected-(U2-I2-Pad7) -> Net-(Q11-C)
- U2 pad 8: unconnected-(U2-I1-Pad8) -> Net-(Q12-C)
- U2 pad 9: unconnected-(U2-I0-Pad9) -> Net-(Q13-C)
- U3 pad 10: unconnected-(U3-9-Pad10) -> LED_IO
- U3 pad 11: unconnected-(U3-10-Pad11) -> MUX_COM2
- U3 pad 2: MUX_COM2 -> S2
- U3 pad 3: S0 -> S3
- U3 pad 4: S1 -> S0
- U3 pad 5: S2 -> S1
- U3 pad 6: S3 -> unconnected-(U3-5-Pad6)
- U3 pad 9: LED_IO -> unconnected-(U3-8-Pad9)
Routing:
- net GND: track 33.6 -> 236.1 mm, vias 0 -> 10
- net Net-(Q33-D): track 62.6 -> 147.1 mm
- net S2: track 0.00 -> 82.1 mm, vias 0 -> 4
- net S3: track 0.00 -> 77.2 mm, vias 0 -> 4
- net 3v3: track 67.9 -> 143.8 mm, vias 32 -> 38
- net S0: track 0.00 -> 61.8 mm, vias 0 -> 2
- net S1: track 0.00 -> 55.7 mm, vias 0 -> 2
- net LED_5V: track 73.3 -> 124.0 mm
- net MUX_COM1: track 0.00 -> 42.6 mm
- net Net-(J1-Pin_2): track 0.00 -> 41.9 mm, vias 0 -> 1
- net MUX_COM2: track 0.00 -> 32.5 mm
- net VCC: track 0.00 -> 32.2 mm
- net Net-(J1-Pin_1): track 0.00 -> 26.9 mm
- net Net-(Q18-C): track 4.15 -> 30.4 mm
- net Net-(Q10-C): track 4.15 -> 29.1 mm
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Other:
- board size 140 x 140 mm -> 405 x 147.4 mm
