File: KiCad/Linesensor_Japan_prot1/Linesensor_Japan_prot1.kicad_sch (KiCad schematic)
At the start: 140 parts, among them J1 Conn_01x04_Socket, J2 Conn_01x02_Socket, Q1 Q_Photo_NPN, Q10 Q_Photo_NPN, Q11 Q_Photo_NPN, Q12 Q_Photo_NPN, Q13 Q_Photo_NPN, Q14 Q_Photo_NPN, Q15 Q_Photo_NPN, Q16 Q_Photo_NPN, Q17 Q_Photo_NPN, Q18 Q_Photo_NPN, Q19 Q_Photo_NPN, Q2 Q_Photo_NPN, Q20 Q_Photo_NPN, Q21 Q_Photo_NPN, Q22 Q_Photo_NPN, Q23 Q_Photo_NPN, Q24 Q_Photo_NPN, Q25 Q_Photo_NPN, Q26 Q_Photo_NPN, Q27 Q_Photo_NPN, Q28 Q_Photo_NPN, Q29 Q_Photo_NPN, Q3 Q_Photo_NPN, Q30 Q_Photo_NPN, Q31 Q_Photo_NPN, Q32 Q_Photo_NPN, Q33 Q_NMOS, Q4 Q_Photo_NPN, Q5 Q_Photo_NPN, Q6 Q_Photo_NPN, Q7 Q_Photo_NPN, Q8 Q_Photo_NPN, Q9 Q_Photo_NPN, U1 CD74HC4067SM, U2 CD74HC4067SM

Commit message: ラインセンサーprot1ほぼ完成
Connections:
- net GND: now also Q2.2 (E)
- net LED_IO: now also U3.10 (9); no longer U3.9 (8)
- net MUX_COM2: now also U3.11 (10); no longer U3.2 (1)
- net S0: now also U3.4 (3); no longer U3.3 (2)
- net S1: now also U3.5 (4); no longer U3.4 (3)
- net S2: now also U3.2 (1); no longer U3.5 (4)
- net S3: now also U3.3 (2); no longer U3.6 (5)
- net at Q5.1 (C), R5.2: now also U1.17 (I14)
- net at Q16.1 (C), R16.2: now also U2.3 (I6)
- net at Q6.1 (C), R6.2: now also U1.16 (I15)
- net at Q25.1 (C), R25.2: now also U2.16 (I15)
- net at Q12.1 (C), R12.2: now also U2.8 (I1)
- net at Q19.1 (C), R19.2: now also U2.22 (I9)
- net at Q28.1 (C), R28.2: now also U1.8 (I1)
- net at Q24.1 (C), R24.2: now also U2.17 (I14)
- net at Q21.1 (C), R21.2: now also U2.20 (I11)
- net at Q30.1 (C), R30.2: now also U1.6 (I3)
- net at Q1.1 (C), R1.2: now also U1.3 (I6); no longer U1.4 (I5)
- net at Q3.1 (C), R3.2: now also U1.19 (I12)
- net at Q2.1 (C), R2.2: now also U1.20 (I11); no longer U1.3 (I6)
- net at Q13.1 (C), R13.2: now also U2.9 (I0)
- net at Q9.1 (C), R9.2: now also U1.23 (I8)
- net at Q4.1 (C), R4.2: now also U1.18 (I13)
- net at U1.2 (I7): now also Q26.1 (C), R26.2
- net at U1.21 (I10): now also Q7.1 (C), R7.2
- net at U1.22 (I9): now also Q8.1 (C), R8.2
- net at U1.5 (I4): now also Q31.1 (C), R31.2
- net at U1.7 (I2): now also Q29.1 (C), R29.2
- net at U1.9 (I0): now also Q27.1 (C), R27.2
- net at Q20.1 (C), R20.2: now also U2.21 (I10)
- net at Q23.1 (C), R23.2: now also U2.18 (I13)
- net at Q14.1 (C), R14.2: now also U2.5 (I4)
- net at Q22.1 (C), R22.2: now also U2.19 (I12)
- net at U2.2 (I7): now also Q17.1 (C), R17.2
- net at U2.23 (I8): now also Q18.1 (C), R18.2
- net at U2.4 (I5): now also Q15.1 (C), R15.2
- net at U2.6 (I3): now also Q10.1 (C), R10.2
- net at U2.7 (I2): now also Q11.1 (C), R11.2
- net at Q32.1 (C), R32.2: now also U1.4 (I5)
Other:
- moved on the sheet: Q1, Q10, Q11, Q12, Q13, Q14, Q15, Q16, Q17, Q18, Q19, Q2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
