File: KiCad/matudachi_motor_prot1/v2_MotorDriver/v2_MotorDriver/v2_MotorDriver.kicad_pcb (KiCad board)
At the start: 2 copper layers, 52.1 x 54.3 mm, 38 parts, among them J6 Conn_01x04_Socket, M1 Conn_01x02_Socket, M2 Conn_01x02_Socket, M3 Conn_01x02_Socket, M4 Conn_01x02_Socket

Commit message: prot2ほぼ完成
Parts:
- added G***: LOGO, JLCPCB_Logos:JCLPCB_30mm, F.Cu at (119.3, 108.7)
