File: KiCad/Linesensor_Japan_prot2/Linesensor_Japan_prot2.kicad_sch (KiCad schematic)
At the start: 152 parts, among them J1 Conn_01x04_Socket, J2 Conn_01x02_Socket, J3 Conn_01x09_Socket, J4 Conn_01x09_Socket, Q1 Q_Photo_NPN, Q10 Q_Photo_NPN, Q11 Q_Photo_NPN, Q12 Q_Photo_NPN, Q13 Q_Photo_NPN, Q14 Q_Photo_NPN, Q15 Q_Photo_NPN, Q16 Q_Photo_NPN, Q17 Q_Photo_NPN, Q18 Q_Photo_NPN, Q19 Q_Photo_NPN, Q2 Q_Photo_NPN, Q20 Q_Photo_NPN, Q21 Q_Photo_NPN, Q22 Q_Photo_NPN, Q23 Q_Photo_NPN, Q24 Q_Photo_NPN, Q25 Q_Photo_NPN, Q26 Q_Photo_NPN, Q27 Q_Photo_NPN, Q28 Q_Photo_NPN, Q29 Q_Photo_NPN, Q3 Q_Photo_NPN, Q30 Q_Photo_NPN, Q31 Q_Photo_NPN, Q32 Q_Photo_NPN, Q33 Q_NMOS, Q4 Q_Photo_NPN, Q5 Q_Photo_NPN, Q6 Q_Photo_NPN, Q7 Q_Photo_NPN, Q8 Q_Photo_NPN, Q9 Q_Photo_NPN, U1 CD74HC4067SM, U2 CD74HC4067SM

Commit message: ああああああああああああああああああ
Parts:
- added D34: D_Schottky, Diode_SMD:D_SOD-323F, symbol Device:D_Schottky
Connections:
- net LED_5V: now also D34.2 (A); no longer D1.2 (A), D10.2 (A), D11.2 (A), D12.2 (A), D13.2 (A), D14.2 (A), D15.2 (A), D16.2 (A), D17.2 (A), D18.2 (A), D19.2 (A), D2.2 (A), D20.2 (A), D21.2 (A), D22.2 (A), D23.2 (A), D24.2 (A), D25.2 (A), D26.2 (A), D27.2 (A), D28.2 (A), D29.2 (A), D3.2 (A), D30.2 (A), D31.2 (A), D32.2 (A), D4.2 (A), D5.2 (A), D6.2 (A), D7.2 (A), D8.2 (A), D9.2 (A)
- new net: D1.2 (A), D10.2 (A), D11.2 (A), D12.2 (A), D13.2 (A), D14.2 (A), D15.2 (A), D16.2 (A), D17.2 (A), D18.2 (A), D19.2 (A), D2.2 (A), D20.2 (A), D21.2 (A), D22.2 (A), D23.2 (A), D24.2 (A), D25.2 (A), D26.2 (A), D27.2 (A), D28.2 (A), D29.2 (A), D3.2 (A), D30.2 (A), D31.2 (A), D32.2 (A), D34.1 (K), D4.2 (A), D5.2 (A), D6.2 (A), D7.2 (A), D8.2 (A), D9.2 (A)
Changed lines of the file:
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@@
 	)
 	(junction
+		(at 121.92 208.28)
+		(diameter 0)
+		(color 0 0 0 0)
+	)
+	(junction
 		(at 383.54 190.5)
 		(diameter 0)
@@
 	)
 	(junction
+		(at 121.92 259.08)
+		(diameter 0)
+		(color 0 0 0 0)
+	)
+	(junction
 		(at 287.02 259.08)
 		(diameter 0)
@@
 	)
 	(junction
+		(at 116.84 208.28)
+		(diameter 0)
+		(color 0 0 0 0)
+	)
+	(junction
 		(at 377.19 36.83)
 		(diameter 0)
@@
 	(wire
 		(pts
+			(xy 116.84 259.08) (xy 121.92 259.08)
+		)
+		(stroke
+			(width 0)
+			(type default)
+		)
+	)
+	(wire
+		(pts
 			(xy 427.99 36.83) (xy 453.39 36.83)
 		)
@@
 	(wire
 		(pts
+			(xy 116.84 208.28) (xy 116.84 259.08)
+		)
+		(stroke
+			(width 0)
+			(type default)
+		)
+	)
+	(wire
+		(pts
 			(xy 690.88 60.96) (xy 690.88 26.67)
 		)
@@
 	(wire
 		(pts
+			(xy 115.57 208.28) (xy 116.84 208.28)
+		)
+		(stroke
+			(width 0)
+			(type default)
+		)
+	)
+	(wire
+		(pts
 			(xy 299.72 274.32) (xy 312.42 274.32)
 		)
@@
 	(wire
 		(pts
+			(xy 116.84 208.28) (xy 121.92 208.28)
+		)
+		(stroke
+			(width 0)
+			(type default)
+		)
+	)
+	(wire
+		(pts
 			(xy 469.9 88.9) (xy 469.9 26.67)
 		)
@@
 		)
 	)
-	(global_label "LED_5V"
-		(shape bidirectional)
-		(at 121.92 259.08 180)
-		(fields_autoplaced yes)
-		(effects
-			(font
-				(size 1.27 1.27)
-			)
-			(justify right)
-		)
-		(property "Intersheetrefs" "${INTERSHEET_REFS}"
-			(at 111.1107 259.08 0)
-			(effects
-				(font
-					(size 1.27 1.27)
-				)
-				(justify right)
-				(hide yes)
-			)
-		)
-		(property "LED_5V" ""
-			(at 121.92 261.2708 0)
-			(effects
-				(font
-					(size 1.27 1.27)
-				)
-				(justify right)
-				(hide yes)
-			)
-		)
-	)
 	(global_label "S2"
 		(shape bidirectional)
@@
 	(global_label "LED_5V"
 		(shape bidirectional)
-		(at 121.92 208.28 180)
+		(at 107.95 208.28 180)
 		(fields_autoplaced yes)
 		(effects
@@
 		)
 		(property "Intersheetrefs" "${INTERSHEET_REFS}"
-			(at 111.1107 208.28 0)
+			(at 97.1407 208.28 0)
 			(effects
 				(font
@@
 		)
 		(property "LED_5V" ""
-			(at 121.92 210.4708 0)
+			(at 107.95 210.4708 0)
 			(effects
 				(font
@@
 					(unit 1)
 				)
+			)
+		)
+	)
+	(symbol
+		(lib_id "Device:D_Schottky")
+		(at 111.76 208.28 180)
+		(unit 1)
+		(exclude_from_sim no)
+		(in_bom yes)
+		(on_board yes)
+		(dnp no)
+		(fields_autoplaced yes)
+		(property "Reference" "D34"
+			(at 112.0775 201.93 0)
+			(effects
+				(font
+					(size 1.27 1.27)
+				)
+			)
+		)
+		(property "Value" "D_Schottky"
+			(at 112.0775 204.47 0)
+			(effects
+				(font
+					(size 1.27 1.27)
+				)
+			)
+		)
+		(property "Footprint" "Diode_SMD:D_SOD-323F"
+			(at 111.76 208.28 0)
+			(effects
+				(font
+					(size 1.27 1.27)
+				)
+				(hide yes)
+			)
+		)
+		(property "Datasheet" "~"
+			(at 111.76 208.28 0)
+			(effects
+				(font
+					(size 1.27 1.27)
+				)
+				(hide yes)
+			)
+		)
+		(property "Description" "Schottky diode"
+			(at 111.76 208.28 0)
+			(effects
+				(font
+					(size 1.27 1.27)
+				)
+				(hide yes)
+			)
+		)
+		(pin "1"
+		)
+		(pin "2"
+		)
+		(instances
+			(project ""
+				(path "/95e5dcf1-74db-4868-be8c-b5f50bcdf3f5"
+					(reference "D34")
+					(unit 1)
+				)

Commit message: IR配置ほぼ完了
Parts:
- J4: footprint Connector_JST:JST_XH_S9B-XH-A-1_1x09_P2.50mm_Horizontal -> Connector_JST2:JST_PH_S9B-PH-K_1x09_P2.00mm_Horizontal
Other:
- note added: "１００ｋ"
Changed lines of the file:
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@@
 		)
 	)
+	(text "１００ｋ"
+		(exclude_from_sim no)
+		(at 94.234 307.34 0)
+		(effects
+			(font
+				(size 1.27 1.27)
+			)
+		)
+	)
 	(text "0.1uF"
 		(exclude_from_sim no)
@@
 			)
 		)
-		(property "Footprint" "Connector_JST:JST_XH_S9B-XH-A-1_1x09_P2.50mm_Horizontal"
+		(property "Footprint" "Connector_JST2:JST_PH_S9B-PH-K_1x09_P2.00mm_Horizontal"
 			(at 38.1 107.95 0)
 			(effects
