File: KiCad/IR_Japan_prot1/IR_Japan_prot1.kicad_pcb (KiCad board)
At the start: 2 copper layers, 100 x 100 mm, 64 parts, among them J1 Conn_01x09_Socket, J2 Conn_01x03_Socket, J3 Conn_01x03_Socket, J4 Conn_01x03_Socket, J5 Conn_01x03_Socket, J6 Conn_01x04_Socket, J7 Conn_01x04_Socket, J8 Conn_01x04_Socket, J9 Conn_01x03_Socket, SW1 SW_DPST_x2, U1 TSSP58038, U10 TSSP58038, U11 TSSP58038, U12 TSSP58038, U13 TSSP58038, U14 TSSP58038, U15 TSSP58038, U16 TSSP58038, U18 CD74HC4067SM, U2 TSSP58038, U3 TSSP58038, U4 TSSP58038, U5 TSSP58038, U6 TSSP58038, U7 TSSP58038, U8 TSSP58038, U9 TSSP58038

Commit message: まると
Parts:
- C1, C10, C11, C12, C13, C14, C15, C16, C2, C3, C4, C5, C6, C7, C8, C9, R1, R10, R11, R12, R13, R14, R15, R16, R2, R3, R4, R5, R6, R7, R8, R9: moved to F.Cu
- moved R12 273.9 mm to (178.4, 139.3), turned to 0 degrees
- moved R13 265.7 mm to (182.9, 118.8), turned to 0 degrees
- moved R14 265.7 mm to (182.9, 121.3), turned to 0 degrees
- moved R15 265.7 mm to (182.9, 123.8), turned to 0 degrees
- moved R16 265.7 mm to (182.9, 126.3), turned to 0 degrees
- moved R3 265.6 mm to (174.3, 138.1), turned to 0 degrees
- moved R10 257.3 mm to (178.5, 133.8), turned to 0 degrees
- moved R11 257.3 mm to (178.5, 136.3), turned to 0 degrees
- moved R4 257.3 mm to (178.5, 118.8), turned to 0 degrees
- moved R5 257.3 mm to (178.5, 121.3), turned to 0 degrees
- moved R6 257.3 mm to (178.5, 123.8), turned to 0 degrees
- moved R7 257.3 mm to (178.5, 126.3), turned to 0 degrees
- moved R8 257.3 mm to (178.5, 128.8), turned to 0 degrees
- moved R9 257.3 mm to (178.5, 131.3), turned to 0 degrees
- moved R1 249.6 mm to (174.4, 132.0), turned to 0 degrees
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Connections:
- C14 pad 1: unconnected-(C14-Pad1) -> Net-(C14-Pad1)
- R14 pad 2: unconnected-(R14-Pad2) -> Net-(C14-Pad1)
- U10 pad 3: unconnected-(U10-Vs-Pad3) -> Net-(SW1A-B)
- U11 pad 3: unconnected-(U11-Vs-Pad3) -> Net-(SW1A-B)
- U12 pad 3: unconnected-(U12-Vs-Pad3) -> Net-(SW1A-B)
- U13 pad 3: unconnected-(U13-Vs-Pad3) -> Net-(SW1A-B)
- U14 pad 3: unconnected-(U14-Vs-Pad3) -> Net-(SW1A-B)
- U15 pad 3: unconnected-(U15-Vs-Pad3) -> Net-(SW1A-B)
- U17 pad 10: S1 -> unconnected-(U17-26,DAC_2-Pad10)
- U17 pad 11: S0 -> LED_IO
- U17 pad 13: unconnected-(U17-*12-Pad13) -> S1
- U17 pad 15: unconnected-(U17-13-Pad15) -> S0
- U17 pad 23: unconnected-(U17-*15-Pad23) -> ball_sensor
- U17 pad 36: unconnected-(U17-22,SCL-Pad36) -> S2
- U17 pad 37: unconnected-(U17-23,MOSI-Pad37) -> S3
- U17 pad 8: S3 -> side_left
- U17 pad 9: S2 -> side_right
- U3 pad 3: GND -> Net-(SW1A-B)
- U4 pad 3: unconnected-(U4-Vs-Pad3) -> Net-(SW1A-B)
- U5 pad 3: unconnected-(U5-Vs-Pad3) -> Net-(SW1A-B)
- U6 pad 3: unconnected-(U6-Vs-Pad3) -> Net-(SW1A-B)
- U7 pad 3: unconnected-(U7-Vs-Pad3) -> Net-(SW1A-B)
- U8 pad 3: unconnected-(U8-Vs-Pad3) -> Net-(SW1A-B)
- U9 pad 3: unconnected-(U9-Vs-Pad3) -> Net-(SW1A-B)
Routing:
- net ball_sensor: track 24.5 -> 105.6 mm, vias 0 -> 1
- net S2: track 8.62 -> 87.6 mm, vias 0 -> 4
- net S3: track 9.05 -> 86.5 mm, vias 0 -> 4
- net GND: track 59.5 -> 101.3 mm, vias 0 -> 3
- net 3v3: track 60.4 -> 82.0 mm, vias 0 -> 1
- net S0: track 7.82 -> 28.6 mm, vias 0 -> 1
- net IR_COM: track 0.00 -> 17.8 mm, vias 0 -> 1
- net S1: track 8.24 -> 23.1 mm, vias 0 -> 1
- net side_right: track 18.1 -> 31.2 mm, vias 0 -> 1
- net side_left: track 12.4 -> 24.7 mm, vias 0 -> 1
- net LED_IO: track 0.00 -> 11.8 mm
- net Net-(SW1A-B): track 0.00 -> 2.65 mm
- net MUX_COM2: track 15.3 -> 16.7 mm
- net TX1(18): track 57.2 -> 57.9 mm
- net RX1(19): track 62.2 -> 62.9 mm
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