File: KiCad/IR_Japan_prot1/メインの穴付き.kicad_pcb (KiCad board)
At the start: 2 copper layers, 100 x 100 mm, 64 parts, among them J1 Conn_01x09_Socket, J2 Conn_01x03_Socket, J3 Conn_01x03_Socket, J4 Conn_01x03_Socket, J5 Conn_01x03_Socket, J6 Conn_01x04_Socket, J7 Conn_01x04_Socket, J8 Conn_01x04_Socket, J9 Conn_01x03_Socket, SW1 SW_DPST_x2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

Commit message: IR配線仕上げ前
Parts:
- removed U18: CD74HC4067SM, Package_SO:SSOP-24_5.3x8.2mm_P0.65mm
- moved C1 0.71 mm to (140.1, 97.8)
- moved R1 0.58 mm to (140.0, 102.5)
- moved C2 0.58 mm to (136.2, 82.1)
- moved R6 0.37 mm to (87.2, 61.7)
Routing:
- net GND: track 379.1 -> 164.5 mm, vias 10 -> 3
- net Net-(U18-I8): track 83.8 -> 0.00 mm, vias 1 -> 0
- net Net-(SW1A-B): track 154.2 -> 80.2 mm
- net Net-(U18-I9): track 69.4 -> 0.00 mm, vias 1 -> 0
- net Net-(U18-I10): track 61.6 -> 2.27 mm, vias 1 -> 0
- net Net-(U18-I7): track 54.8 -> 0.00 mm, vias 1 -> 0
- net Net-(U18-I11): track 53.6 -> 0.00 mm, vias 1 -> 0
- net Net-(U18-I15): track 51.6 -> 0.00 mm, vias 1 -> 0
- net Net-(U18-I6): track 49.8 -> 0.00 mm, vias 1 -> 0
- net Net-(U18-I5): track 48.5 -> 0.00 mm, vias 1 -> 0
- net Net-(U18-I12): track 48.1 -> 0.00 mm, vias 1 -> 0
- net Net-(U18-I13): track 46.7 -> 0.00 mm, vias 1 -> 0
- net Net-(U18-I14): track 44.1 -> 0.00 mm, vias 1 -> 0
- net Net-(U18-I1): track 41.9 -> 0.00 mm, vias 1 -> 0
- net Net-(U18-I2): track 40.6 -> 0.00 mm, vias 1 -> 0
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Other:
- outline, holes or cut-outs redrawn
