File: KiCad/IR_Japan_prot1/IR_Japan_prot1.kicad_sch (KiCad schematic)
At the start: 64 parts, among them J1 Conn_01x09_Socket, J2 Conn_01x03_Socket, J3 Conn_01x03_Socket, J4 Conn_01x03_Socket, J5 Conn_01x03_Socket, J6 Conn_01x04_Socket, J7 Conn_01x04_Socket, J8 Conn_01x04_Socket, J9 Conn_01x03_Socket, SW1 SW_DPST_x2, U1 TSSP58038, U10 TSSP58038, U11 TSSP58038, U12 TSSP58038, U13 TSSP58038, U14 TSSP58038, U15 TSSP58038, U16 TSSP58038, U18 CD74HC4067SM, U2 TSSP58038, U3 TSSP58038, U4 TSSP58038, U5 TSSP58038, U6 TSSP58038, U7 TSSP58038, U8 TSSP58038, U9 TSSP58038

Commit message: まると
Connections:
- net GND: no longer U3.3 (Vs)
- net LED_IO: now also U17.11 (27)
- net S0: now also U17.15 (13); no longer U17.11 (27)
- net S1: now also U17.13 (*12); no longer U17.10 (26,DAC_2)
- net S2: now also U17.36 (22,SCL); no longer U17.9 (25,DAC_1)
- net S3: now also U17.37 (23,MOSI)
- net ball_sensor: now also U17.23 (*15)
- net side_left: now also U17.8 (33)
- net side_right: now also U17.9 (25,DAC_1)
- net at SW1.2 (B), U1.3 (Vs), U16.3 (Vs)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: now also U10.3 (Vs), U11.3 (Vs), U12.3 (Vs), U13.3 (Vs), U14.3 (Vs), U15.3 (Vs), U3.3 (Vs), U4.3 (Vs), U5.3 (Vs), U6.3 (Vs), U7.3 (Vs), U8.3 (Vs), U9.3 (Vs)
- net at R14.2: now also C14.1
Other:
- note added: "ADC1 系列 GPIO32 GPIO33 GPIO34（入力専用） GPIO35（入力専用） GPIO36 (SVP)（入力専用） GPIO39 (SVN)（入力専用）"
- note added: "ADC2 GPIO0 GPIO2 GPIO4 GPIO12 GPIO13 GPIO14 GPIO15 GPIO25 GPIO26 GPIO27"
- note added: "PWM GPIO16 GPIO17 GPIO18 GPIO19 GPIO21 GPIO22 GPIO23 GPIO25 GPIO26 GPIO27 GPIO32 GPIO33"

Commit message: IR配線仕上げ前
Connections:
- net at C1.1, R1.2: now also U18.23 (I8)
- net at C11.1, R11.2: now also U18.17 (I14)
- net at C5.1, R5.2: now also U18.5 (I4)
- net at C14.1, R14.2: now also U18.20 (I11)
- net at C9.1, R9.2: now also U18.9 (I0)
- net at C6.1, R6.2: now also U18.6 (I3)
- net at C2.1, R2.2: now also U18.2 (I7)
- net at C16.1, R16.2: now also U18.22 (I9)
- net at C13.1, R13.2: now also U18.19 (I12)
- net at C4.1, R4.2: now also U18.4 (I5)
- net at C3.1, R3.2: now also U18.3 (I6)
- net at C15.1, R15.2: now also U18.21 (I10)
- net at C8.1, R8.2: now also U18.8 (I1)
- net at U18.16 (I15): now also C10.1, R10.2
- net at U18.18 (I13): now also C12.1, R12.2
- net at U18.7 (I2): now also C7.1, R7.2

Commit message: IR完成
Parts:
- added J10: Conn_02x03_Top_Bottom, Connector_PinHeader_2.54mm:PinHeader_2x03_P2.54mm_Vertical, symbol Connector_Generic:Conn_02x03_Top_Bottom
Connections:
- net 3v3: now also J4.1 (Pin_1)
- net at U17.24 (*2): now also J10.6 (Pin_6)
- net at U17.25 (*0): now also J10.4 (Pin_4)
- net at U17.26 (*4): now also J10.5 (Pin_5)
- net at U17.29 (*5,CS): now also J10.3 (Pin_3)
- net at U17.32 (GND): now also J10.1 (Pin_1)
- net at U17.33 (21,SDA): now also J10.2 (Pin_2)

Commit message: IRあと文字
Parts:
- removed J10: Conn_02x03_Top_Bottom, Connector_PinHeader_2.54mm:PinHeader_2x03_P2.54mm_Vertical, symbol Connector_Generic:Conn_02x03_Top_Bottom
- added C17: C, Capacitor_SMD:C_0603_1608Metric_Pad1.08x0.95mm_HandSolder, symbol Device:C
- added C18: C_Polarized_US, Capacitor_THT:C_Radial_D8.0mm_H11.5mm_P3.50mm, symbol Device:C_Polarized_US
- added D1: D_Schottky, Diode_SMD:D_SOD-323_HandSoldering, symbol Device:D_Schottky
- added J11: Conn_02x05_Top_Bottom, Connector_PinHeader_2.54mm:PinHeader_2x05_P2.54mm_Vertical, symbol Connector_Generic:Conn_02x05_Top_Bottom
Connections:
- net 3v3: now also J11.5 (Pin_5)
- net GND: now also C17.2, C18.2, J11.1 (Pin_1)
- net VCC: now also D1.2 (A); no longer U17.19 (5V)
- net at U17.10 (26,DAC_2): now also J11.6 (Pin_6)
- net at U17.12 (*14): now also J11.4 (Pin_4)
- net at U17.24 (*2): now also J11.8 (Pin_8)
- net at U17.25 (*0): now also J11.10 (Pin_10)
- net at U17.26 (*4): now also J11.9 (Pin_9)
- net at U17.29 (*5,CS): now also J11.7 (Pin_7)
- net at U17.33 (21,SDA): now also J11.3 (Pin_3)
- new net: C17.1, C18.1, D1.1 (K), J11.2 (Pin_2), U17.19 (5V)
Other:
- moved on the sheet: C1, C10, C11, C12, C13, C14, C15, C16, C2, C3, C4, C5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

Commit message: IRmadeowari
Parts:
- added J10: Conn_01x02_Socket, Connector_PinHeader_2.54mm:PinHeader_1x02_P2.54mm_Vertical, symbol Connector:Conn_01x02_Socket
Connections:
- net GND: now also J10.1 (Pin_1)
- net VCC: now also J10.2 (Pin_2)
Changed lines of the file:
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@@
 	(wire
 		(pts
+			(xy 83.82 186.69) (xy 96.52 186.69)
+		)
+		(stroke
+			(width 0)
+			(type default)
+		)
+	)
+	(wire
+		(pts
 			(xy 618.49 63.5) (xy 618.49 73.66)
 		)
@@
 	(wire
 		(pts
+			(xy 96.52 186.69) (xy 96.52 185.42)
+		)
+		(stroke
+			(width 0)
+			(type default)
+		)
+	)
+	(wire
+		(pts
 			(xy 504.19 77.47) (xy 529.59 77.47)
 		)
@@
 	(wire
 		(pts
+			(xy 83.82 189.23) (xy 96.52 189.23)
+		)
+		(stroke
+			(width 0)
+			(type default)
+		)
+	)
+	(wire
+		(pts
 			(xy 82.55 223.52) (xy 96.52 223.52)
 		)
@@
 	)
 	(symbol
+		(lib_id "power:VCC")
+		(at 96.52 185.42 0)
+		(unit 1)
+		(exclude_from_sim no)
+		(in_bom yes)
+		(on_board yes)
+		(dnp no)
+		(fields_autoplaced yes)
+		(property "Reference" "#PWR021"
+			(at 96.52 189.23 0)
+			(effects
+				(font
+					(size 1.27 1.27)
+				)
+				(hide yes)
+			)
+		)
+		(property "Value" "VCC"
+			(at 96.52 180.34 0)
+			(effects
+				(font
+					(size 1.27 1.27)
+				)
+			)
+		)
+		(property "Footprint" ""
+			(at 96.52 185.42 0)
+			(effects
+				(font
+					(size 1.27 1.27)
+				)
+				(hide yes)
+			)
+		)
+		(property "Datasheet" ""
+			(at 96.52 185.42 0)
+			(effects
+				(font
+					(size 1.27 1.27)
+				)
+				(hide yes)
+			)
+		)
+		(property "Description" "Power symbol creates a global label with name \"VCC\""
+			(at 96.52 185.42 0)
+			(effects
+				(font
+					(size 1.27 1.27)
+				)
+				(hide yes)
+			)
+		)
+		(pin "1"
+		)
+		(instances
+			(project "IR_Japan_prot1"
+				(path "/265029e8-5ce2-48e4-915a-807e964409e7"
+					(reference "#PWR021")
+					(unit 1)
+				)
+			)
+		)
+	)
+	(symbol
 		(lib_id "Sensor_Proximity:TSSP58038")
 		(at 575.31 53.34 270)
@@
 	)
 	(symbol
+		(lib_id "Connector:Conn_01x02_Socket")
+		(at 78.74 189.23 180)
+		(unit 1)
+		(exclude_from_sim no)
+		(in_bom yes)
+		(on_board yes)
+		(dnp no)
+		(fields_autoplaced yes)
+		(property "Reference" "J10"
+			(at 79.375 181.61 0)
+			(effects
+				(font
+					(size 1.27 1.27)
+				)
+			)
+		)
+		(property "Value" "Conn_01x02_Socket"
+			(at 79.375 184.15 0)
+			(effects
+				(font
+					(size 1.27 1.27)
+				)
+			)
+		)
+		(property "Footprint" "Connector_PinHeader_2.54mm:PinHeader_1x02_P2.54mm_Vertical"
+			(at 78.74 189.23 0)
+			(effects
+				(font
+					(size 1.27 1.27)
+				)
+				(hide yes)
+			)
+		)
+		(property "Datasheet" "~"
+			(at 78.74 189.23 0)
+			(effects
+				(font
+					(size 1.27 1.27)
+				)
+				(hide yes)
+			)
+		)
+		(property "Description" "Generic connector, single row, 01x02, script generated"
+			(at 78.74 189.23 0)
+			(effects
+				(font
+					(size 1.27 1.27)
+				)
+				(hide yes)
+			)
+		)
+		(pin "1"
+		)
+		(pin "2"
+		)
+		(instances
+			(project ""
+				(path "/265029e8-5ce2-48e4-915a-807e964409e7"
+					(reference "J10")
+					(unit 1)
+				)
+			)
+		)
+	)
+	(symbol
 		(lib_id "Device:C")
 		(at 368.3 73.66 270)
@@
 					(unit 1)
 				)
+			)
+		)
+	)
+	(symbol
+		(lib_id "power:GND")
+		(at 96.52 189.23 0)
+		(unit 1)
+		(exclude_from_sim no)
+		(in_bom yes)
+		(on_board yes)
+		(dnp no)
+		(fields_autoplaced yes)
+		(property "Reference" "#PWR022"
+			(at 96.52 195.58 0)
+			(effects
+				(font
+					(size 1.27 1.27)
+				)
+				(hide yes)
+			)
+		)
+		(property "Value" "GND"
+			(at 96.52 194.31 0)
+			(effects
+				(font
+					(size 1.27 1.27)
+				)
+			)
+		)
+		(property "Footprint" ""
+			(at 96.52 189.23 0)
+			(effects
+				(font
+					(size 1.27 1.27)
+				)
+				(hide yes)
+			)
+		)
+		(property "Datasheet" ""
+			(at 96.52 189.23 0)
+			(effects
+				(font
+					(size 1.27 1.27)
+				)
+				(hide yes)
+			)
+		)
+		(property "Description" "Power symbol creates a global label with name \"GND\" , ground"
+			(at 96.52 189.23 0)
+			(effects
+				(font
+					(size 1.27 1.27)
+				)
+				(hide yes)
+			)
+		)
+		(pin "1"
+		)
+		(instances
+			(project "IR_Japan_prot1"
+				(path "/265029e8-5ce2-48e4-915a-807e964409e7"
+					(reference "#PWR022")
+					(unit 1)
+				)
