File: KiCad/tachanka_Main_prot1/RCJ_main/RCJ_main.kicad_sch (KiCad schematic)
At the start: 20 parts, among them J1 Conn_01x02_Socket, J2 Conn_01x03_Socket, J3 Conn_01x02_Socket, U1 RP2040-Zero, U2 ESP32-WROOM-32D

Commit message: あ
Other:
- moved on the sheet: D1, D2, J3, R1, R2
