File: KiCad/Main_RCJ_Japan_prot2/Main_RCJ_Japan_prot2.kicad_pcb (KiCad board)
At the start: 2 copper layers, 99.5 x 94.9 mm, 32 parts, among them J1 Conn_01x04_Socket, J10 Conn_01x02_Socket, J11 Conn_01x03_Socket, J12 Conn_01x03_Socket, J13 Conn_01x02_Socket, J14 Conn_01x02_Socket, J2 Conn_01x04_Socket, J3 Conn_01x04_Socket, J4 Conn_01x04_Socket, J5 Conn_01x04_Socket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

Commit message: 画像インポートクラッシュくそ
Parts:
- moved R1 4.64 mm to (118.1, 143.7)
- moved R2 4.11 mm to (117.0, 139.6)
Connections:
- R2 pad 1: Net-(J10-Pin_1) -> GND
Routing:
- net GND: track 245.9 -> 251.8 mm
- net Net-(J10-Pin_1): track 14.1 -> 9.37 mm
Changed lines of the file:
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@@
 	(footprint "Resistor_THT:R_Axial_DIN0309_L9.0mm_D3.2mm_P12.70mm_Horizontal"
 		(layer "F.Cu")
-		(at 116.91 139.212 180)
+		(at 118.1 143.7 180)
 		(descr "Resistor, Axial_DIN0309 series, Axial, Horizontal, pin pitch=12.7mm, 0.5W = 1/2W, length*diameter=9*3.2mm^2, http://cdn-reichelt.de/documents/datenblatt/B400/1_4W%23YAG.pdf")
 		(tags "Resistor Axial_DIN0309 series Axial Horizontal pin pitch 12.7mm 0.5W = 1/2W length 9mm diameter 3.2mm")
@@
 	(footprint "Resistor_THT:R_Axial_DIN0309_L9.0mm_D3.2mm_P12.70mm_Horizontal"
 		(layer "F.Cu")
-		(at 118.269 143.46 180)
+		(at 117 139.55 180)
 		(descr "Resistor, Axial_DIN0309 series, Axial, Horizontal, pin pitch=12.7mm, 0.5W = 1/2W, length*diameter=9*3.2mm^2, http://cdn-reichelt.de/documents/datenblatt/B400/1_4W%23YAG.pdf")
 		(tags "Resistor Axial_DIN0309 series Axial Horizontal pin pitch 12.7mm 0.5W = 1/2W length 9mm diameter 3.2mm")
@@
 			(layers "*.Cu" "*.Mask")
 			(remove_unused_layers no)
-			(net 34 "Net-(J10-Pin_1)")
+			(net 6 "GND")
 			(pintype "passive")
 		)
@@
 	)
 	(segment
+		(start 117 139.55)
+		(end 120.296 139.55)
+		(width 2)
+		(layer "F.Cu")
+		(net 6)
+	)
+	(segment
 		(start 104.84 137.729)
 		(end 122.117 137.729)
@@
 	)
 	(segment
+		(start 120.296 139.55)
+		(end 122.117 137.729)
+		(width 2)
+		(layer "F.Cu")
+		(net 6)
+	)
+	(segment
 		(start 100.313 133.202)
 		(end 98.42 135.095)
@@
 	)
 	(segment
+		(start 105.4 143.7)
+		(end 105.4 140.65)
+		(width 2)
+		(layer "F.Cu")
+		(net 9)
+	)
+	(segment
 		(start 86.32492 124.06745)
 		(end 86.999735 124.742265)
@@
 		(net 9)
 	)
+	(segment
+		(start 105.4 140.65)
+		(end 104.3 139.55)
+		(width 2)
+		(layer "F.Cu")
+		(net 9)
+	)
 	(via
 		(at 86.999735 124.742265)
@@
 	)
 	(segment
-		(start 91.746 132.742)
-		(end 96.744 137.74)
+		(start 98.554 139.55)
+		(end 104.3 139.55)
 		(width 0.2)
 		(layer "B.Cu")
@@
 	)
 	(segment
-		(start 105.569 140.571)
-		(end 104.21 139.212)
-		(width 2)
-		(layer "B.Cu")
-		(net 9)
-	)
-	(segment
 		(start 85.408 89.929)
 		(end 84.971 90.366)
@@
 	)
 	(segment
-		(start 105.569 143.46)
-		(end 105.569 140.571)
-		(width 2)
-		(layer "B.Cu")
-		(net 9)
-	)
-	(segment
-		(start 102.738 137.74)
-		(end 104.21 139.212)
-		(width 0.2)
-		(layer "B.Cu")
-		(net 9)
-	)
-	(segment
-		(start 91.746 129.48853)
-		(end 91.746 132.742)
-		(width 0.2)
-		(layer "B.Cu")
-		(net 9)
-	)
-	(segment
-		(start 96.744 137.74)
-		(end 102.738 137.74)
+		(start 91.746 132.742)
+		(end 98.554 139.55)
 		(width 0.2)
 		(layer "B.Cu")
@@
 	)
 	(segment
+		(start 91.746 129.48853)
+		(end 91.746 132.742)
+		(width 0.2)
+		(layer "B.Cu")
+		(net 9)
+	)
+	(segment
 		(start 84.971 107.527)
 		(end 84.971 113.761)
@@
 	)
 	(segment
-		(start 118.269 143.46)
-		(end 118.269 140.571)
-		(width 2)
-		(layer "B.Cu")
-		(net 34)
-	)
-	(segment
 		(start 124.617 137.729)
-		(end 124.617 138.729)
+		(end 124.617 138.383)
 		(width 2)
-		(layer "B.Cu")
-		(net 34)
-	)
-	(segment
-		(start 124.617 138.729)
-		(end 119.886 143.46)
-		(width 2)
-		(layer "B.Cu")
+		(layer "F.Cu")
 		(net 34)
 	)
 	(segment
-		(start 118.269 140.571)
-		(end 116.91 139.212)
+		(start 124.617 138.383)
+		(end 119.3 143.7)
 		(width 2)
-		(layer "B.Cu")
+		(layer "F.Cu")
 		(net 34)
 	)
 	(segment
-		(start 119.886 143.46)
-		(end 118.269 143.46)
+		(start 119.3 143.7)
+		(end 118.1 143.7)
 		(width 2)
-		(layer "B.Cu")
+		(layer "F.Cu")
 		(net 34)
 	)
